File: Kicad/DK60TP.sch (KiCad schematic (older format))
At the start: 21 parts, among them J1 USB_mini_micro_B, M1 MISC, M2 MISC, M3 MISC, M4 MISC, P1 MOUSE_BOARD, SW1 SW_PUSH, U0 ATMEGA32U4, X1 XTAL_GND

Commit message: - Updated routing
Connections:
- net Col6: now also U0.25 (ICP1/PD4); no longer U0.26 (T1/PD6)
- net Col8: now also U0.26 (T1/PD6); no longer U0.25 (ICP1/PD4)
Changed lines of the file:
@@
 Text GLabel 4650 1350 2    60   Input ~ 0
 Col2
-Text GLabel 4650 2650 2    60   Input ~ 0
+Text GLabel 4650 2750 2    60   Input ~ 0
 Col6
 Text GLabel 2500 1850 0    60   Input ~ 0
 Col7
-Text GLabel 4650 2750 2    60   Input ~ 0
+Text GLabel 4650 2650 2    60   Input ~ 0
 Col8
 Text GLabel 4650 2450 2    60   Input ~ 0

Commit message: - FIxed bug in wiring (missing connections)
Connections:
- net GND: now also X1.3
Changed lines of the file:
@@
 	7650 4400 7650 4300
 Wire Wire Line
-	7200 4450 7200 4400
+	7200 4200 7200 4450
 Connection ~ 7200 4400
 Wire Notes Line

Commit message: - First draw for Rev. B
Parts:
- removed M3, M4: MISC, Footprint:BreakHoles, symbol MISC
- U0: value ATMEGA32U4 -> ATMEGA32U4-MU; footprint Housings_QFP:TQFP-44_10x10mm_Pitch0.8mm -> Housings_DFN_QFN:QFN-44-1EP_7x7mm_Pitch0.5mm
Connections:
- net Col5: now also U0.8 (PB0/SS); no longer U0.9 (PB1/SCK)
- net Col6: now also U0.10 (PB2/MOSI); no longer U0.25 (ICP1/PD4)
- net ColD: now also U0.25 (ICP1/PD4); no longer U0.8 (PB0/SS)
- net Row3: now also U0.9 (PB1/SCK); no longer U0.10 (PB2/MOSI)
Changed lines of the file:
@@
 P 3550 1900
 F 0 "U0" H 3550 650 60  0001 C CNN
-F 1 "ATMEGA32U4" H 3550 3150 60  0001 C CNN
-F 2 "Housings_QFP:TQFP-44_10x10mm_Pitch0.8mm" H 3550 1900 60  0001 C CNN
+F 1 "ATMEGA32U4-MU" H 3550 3150 60  0001 C CNN
+F 2 "Housings_DFN_QFN:QFN-44-1EP_7x7mm_Pitch0.5mm" H 3550 1900 60  0001 C CNN
 F 3 "" H 3550 1900 60  0000 C CNN
 	1    3550 1900
@@
 F10 "RGB" I R 6800 2000 60
 $EndSheet
-Text GLabel 2500 1650 0    60   Input ~ 0
+Text GLabel 2500 1550 0    60   Input ~ 0
 Col5
 Text GLabel 4650 2250 2    60   Input ~ 0
@@
 Text GLabel 4650 1350 2    60   Input ~ 0
 Col2
-Text GLabel 4650 2750 2    60   Input ~ 0
+Text GLabel 2500 1750 0    60   Input ~ 0
 Col6
 Text GLabel 2500 1850 0    60   Input ~ 0
@@
 Text GLabel 2500 2550 0    60   Input ~ 0
 ColC
-Text GLabel 2500 1550 0    60   Input ~ 0
+Text GLabel 4650 2750 2    60   Input ~ 0
 ColD
 Text GLabel 4650 1550 2    60   Input ~ 0
@@
 Text GLabel 4650 2350 2    60   Input ~ 0
 Row2
-Text GLabel 2500 1750 0    60   Input ~ 0
+Text GLabel 2500 1650 0    60   Input ~ 0
 Row3
 $Comp
@@
 $EndComp
 $Comp
-L MISC M3
-U 1 1 593CCFFA
-P 1250 3950
-F 0 "M3" H 1250 4100 60  0000 C CNN
-F 1 "MISC" H 1250 3800 60  0000 C CNN
-F 2 "Footprint:BreakHoles" H 1250 3950 60  0001 C CNN
-F 3 "" H 1250 3950 60  0000 C CNN
-	1    1250 3950
-	1    0    0    -1
-$EndComp
-$Comp
-L MISC M2
-U 1 1 593CD07A
-P 900 4400
-F 0 "M2" H 900 4550 60  0000 C CNN
-F 1 "MISC" H 900 4250 60  0000 C CNN
-F 2 "Footprint:BreakHoles" H 900 4400 60  0001 C CNN
-F 3 "" H 900 4400 60  0000 C CNN
-	1    900  4400
-	1    0    0    -1
-$EndComp
-$Comp
-L MISC M4
-U 1 1 593CD101
-P 1250 4400
-F 0 "M4" H 1250 4550 60  0000 C CNN
-F 1 "MISC" H 1250 4250 60  0000 C CNN
-F 2 "Footprint:BreakHoles" H 1250 4400 60  0001 C CNN
-F 3 "" H 1250 4400 60  0000 C CNN
-	1    1250 4400
-	1    0    0    -1
-$EndComp
-$Comp
 L VCC #PWR015
 U 1 1 593CBBEA
@@
 Text Label 5600 4250 0    60   ~ 0
 RGB_TP
+$Comp
+L MISC M2
+U 1 1 59F15D36
+P 1300 3950
+F 0 "M2" H 1300 4100 60  0000 C CNN
+F 1 "MISC" H 1300 3800 60  0000 C CNN
+F 2 "Footprint:BreakHoles" H 1300 3950 60  0001 C CNN
+F 3 "" H 1300 3950 60  0000 C CNN
+	1    1300 3950
+	1    0    0    -1
+$EndComp
 $EndSCHEMATC

Commit message: - Updated ATMEGA to MU version
Connections:
- net GND: now also U0.45 (GND)
Other:
- moved on the sheet: C1, C2, C3, C4, C5, C6, C7, M1, M2, P1, R1, SW1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

Commit message: - Updated ATMEGA controller (AU and MU package)
Parts:
- U0: symbol ATMEGA32U4 -> ATMEGA32U4-MU
Changed lines of the file:
@@
 EESchema Schematic File Version 2
 LIBS:power
-LIBS:device
-LIBS:transistors
-LIBS:conn
-LIBS:linear
-LIBS:regul
-LIBS:74xx
-LIBS:cmos4000
-LIBS:adc-dac
-LIBS:memory
-LIBS:xilinx
-LIBS:microcontrollers
-LIBS:dsp
-LIBS:microchip
-LIBS:analog_switches
-LIBS:motorola
-LIBS:texas
-LIBS:intel
-LIBS:audio
-LIBS:interface
-LIBS:digital-audio
-LIBS:philips
-LIBS:display
-LIBS:cypress
-LIBS:siliconi
-LIBS:opto
-LIBS:atmel
-LIBS:contrib
-LIBS:valves
-LIBS:keyboard_parts
-LIBS:mkl27z256vfm4
-LIBS:TS65
 LIBS:DK60TP-cache
 EELAYER 25 0
@@
 $EndComp
 $Comp
-L ATMEGA32U4 U0
+L ATMEGA32U4-MU U0
 U 1 1 591F6C9B
 P 3550 1900

Commit message: - Simplifying routage (1 over n)
Connections:
- net at U0.4 (D+): now also R4.1; no longer R4.2
- net at J1.3 (D+): now also R4.2; no longer R4.1
Changed lines of the file:
@@
 F 3 "" H 1600 1150 50  0001 C CNN
 	1    1600 1150
-	0    -1   -1   0
+	0    1    1    0
 $EndComp
 $Comp

Commit message: - Simplifying routing (3/n)
Parts:
- M1, M2: footprint Footprint:BreakHoles -> Footprint:BreakHoles_small
Changed lines of the file:
@@
 F 0 "M1" H 900 4450 60  0000 C CNN
 F 1 "MISC" H 900 4150 60  0000 C CNN
-F 2 "Footprint:BreakHoles" H 900 4300 60  0001 C CNN
+F 2 "Footprint:BreakHoles_small" H 900 4300 60  0001 C CNN
 F 3 "" H 900 4300 60  0000 C CNN
 	1    900  4300
@@
 F 0 "M2" H 1300 4450 60  0000 C CNN
 F 1 "MISC" H 1300 4150 60  0000 C CNN
-F 2 "Footprint:BreakHoles" H 1300 4300 60  0001 C CNN
+F 2 "Footprint:BreakHoles_small" H 1300 4300 60  0001 C CNN
 F 3 "" H 1300 4300 60  0000 C CNN
 	1    1300 4300
