File: Kicad/DK60TP.sch (KiCad schematic (older format))
At the start: 19 parts, among them J1 USB_mini_micro_B, M1 MISC, M2 MISC, P1 MOUSE_BOARD, SW1 RESET, U0 ATMEGA32U4-MU, Y1 Crystal

Commit message: - Updated som manf# for mouser
Parts:
- J1: manf# 609-4618-1-ND -> 105017-0001
- R1, R2: manf# RMCF0805JT10K0 -> CR0805-JW-103ELF
- R3, R4: manf# RMCF0805JT22R0 -> CR0805-JW-220ELF
Changed lines of the file:
@@
 F 1 "10K" V 3500 4250 50  0000 C CNN
 F 2 "Resistors_SMD:R_0805_HandSoldering" V 3430 4250 50  0001 C CNN
-F 3 "https://www.seielect.com/Catalog/SEI-RMCF_RMCP.pdf" H 3500 4250 50  0001 C CNN
-F 4 "RMCF0805JT10K0" V 3500 4250 60  0001 C CNN "manf#"
+F 3 "http://www.mouser.com/ds/2/54/chpreztr-977002.pdf" H 3500 4250 50  0001 C CNN
+F 4 "CR0805-JW-103ELF" V 3500 4250 60  0001 C CNN "manf#"
 	1    3500 4250
 	0    -1   -1   0
@@
 F 1 "10K" V 5150 2300 50  0000 C CNN
 F 2 "Resistors_SMD:R_0805_HandSoldering" V 5080 2300 50  0001 C CNN
-F 3 "https://www.seielect.com/Catalog/SEI-RMCF_RMCP.pdf" H 5150 2300 50  0001 C CNN
-F 4 "RMCF0805JT10K0" V 5150 2300 60  0001 C CNN "manf#"
+F 3 "http://www.mouser.com/ds/2/54/chpreztr-977002.pdf" H 5150 2300 50  0001 C CNN
+F 4 "CR0805-JW-103ELF" V 5150 2300 60  0001 C CNN "manf#"
 	1    5150 2300
 	-1   0    0    1
@@
 F 1 "USB_mini_micro_B" H 950 1350 60  0001 C CNN
 F 2 "Footprint:Micro_USB_Hand" H 1050 1100 60  0001 C CNN
-F 3 "http://portal.fciconnect.com/Comergent//fci/drawing/10118194.pdf" H 1050 1100 60  0001 C CNN
-F 4 "609-4618-1-ND" H 1100 1100 60  0001 C CNN "manf#"
+F 3 "http://www.mouser.com/ds/2/276/1050170001_IO_CONNECTORS-230168.pdf" H 1050 1100 60  0001 C CNN
+F 4 "105017-0001" H 1100 1100 60  0001 C CNN "manf#"
 	1    1100 1100
 	1    0    0    -1
@@
 F 1 "22" V 1950 1050 50  0000 C CNN
 F 2 "Resistors_SMD:R_0805_HandSoldering" V 1880 1050 50  0001 C CNN
-F 3 "https://www.seielect.com/Catalog/SEI-RMCF_RMCP.pdf" H 1950 1050 50  0001 C CNN
-F 4 "RMCF0805JT22R0" V 1950 1050 60  0001 C CNN "manf#"
+F 3 "http://www.mouser.com/ds/2/54/chpreztr-977002.pdf" H 1950 1050 50  0001 C CNN
+F 4 "CR0805-JW-220ELF" V 1950 1050 60  0001 C CNN "manf#"
 	1    1950 1050
 	0    1    1    0
@@
 F 1 "22" V 1600 1150 50  0000 C CNN
 F 2 "Resistors_SMD:R_0805_HandSoldering" V 1530 1150 50  0001 C CNN
-F 3 "https://www.seielect.com/Catalog/SEI-RMCF_RMCP.pdf" H 1600 1150 50  0001 C CNN
-F 4 "RMCF0805JT22R0" V 1600 1150 60  0001 C CNN "manf#"
+F 3 "http://www.mouser.com/ds/2/54/chpreztr-977002.pdf" H 1600 1150 50  0001 C CNN
+F 4 "CR0805-JW-220ELF" V 1600 1150 60  0001 C CNN "manf#"
 	1    1600 1150
 	0    1    1    0

Commit message: Updated wiring
Swap RGB and Row4 pins
Changed lines of the file:
@@
 EESchema Schematic File Version 2
 LIBS:kicad_parts
+LIBS:DK60TP-cache
 EELAYER 25 0
 EELAYER END
@@
 Text GLabel 4650 1650 2    60   Input ~ 0
 Col3
-Text GLabel 4650 2650 2    60   Input ~ 0
+Text GLabel 4650 2550 2    60   Input ~ 0
 Row4
 Text GLabel 4650 2450 2    60   Input ~ 0
@@
 F1 "HOLES.sch" 60
 $EndSheet
-Text GLabel 4650 2550 2    60   Input ~ 0
+Text GLabel 4650 2650 2    60   Input ~ 0
 RGB
 $Comp

Commit message: Less than 100 VIAs!
Inverted col8 and col9 on Atmega to reduce the quantity of VIAs.
Changed lines of the file:
@@
 Text GLabel 2500 1850 0    60   Input ~ 0
 Col7
+Text GLabel 4650 1250 2    60   Input ~ 0
+Col8
 Text GLabel 4650 1350 2    60   Input ~ 0
-Col8
-Text GLabel 4650 1250 2    60   Input ~ 0
 Col9
 Text GLabel 2500 2850 0    60   Input ~ 0

Commit message: Added 2 break holes and updated renders
* Added 2 break holes to increase solidity in case of the user wont
seperate the 2 parts
* Removed some 3D Shape to have a better render view
Parts:
- added M3, M4: MISC, Footprint:BreakHoles_small, symbol MISC
Changed lines of the file:
@@
 Wire Wire Line
 	7200 4750 7200 4800
+$Comp
+L MISC M3
+U 1 1 59F5B977
+P 900 4750
+F 0 "M3" H 900 4900 60  0000 C CNN
+F 1 "MISC" H 900 4600 60  0000 C CNN
+F 2 "Footprint:BreakHoles_small" H 900 4750 60  0001 C CNN
+F 3 "" H 900 4750 60  0000 C CNN
+	1    900  4750
+	1    0    0    -1
+$EndComp
+$Comp
+L MISC M4
+U 1 1 59F5BA24
+P 1300 4750
+F 0 "M4" H 1300 4900 60  0000 C CNN
+F 1 "MISC" H 1300 4600 60  0000 C CNN
+F 2 "Footprint:BreakHoles_small" H 1300 4750 60  0001 C CNN
+F 3 "" H 1300 4750 60  0000 C CNN
+	1    1300 4750
+	1    0    0    -1
+$EndComp
 $EndSCHEMATC
