File: Kicad/MATRIX.sch (KiCad schematic (older format))
At the start: 148 parts, among them K1 K00, K10 K11, K11 K21, K12 K31, K13 K41, K14 K41, K15 K02, K16 K12, K17 K22, K18 K32, K19 K42, K2 K10, K20 K42, K21 K03, K22 K13, K23 K23, K24 K33, K25 K2D, K26 K3D, K27 K04, K28 K14, K29 K24, K3 K20, K30 K34, K31 K3C, K32 K05, K33 K15, K34 K25, K35 K35, K38 K06, K39 K16, K4 K20, K40 K26, K41 K36, K42 K46, K44 K46, K45 K46, K46 K07, K47 K17, K48 K27, K49 K37, K5 K30, K50 K08, K51 K18, K52 K28, K53 K38, K54 K09, K55 K19, K56 K29, K57 K39, K58 K49, K59 K0A, K6 K30, K60 K1A, K61 K2A, K62 K3A, K63 K4A, K64 K4A, K65 K0B, K66 K1B, K67 K2B, K68 K3B, K69 K4B, K7 K40, K70 K4B, K71 K4B, K72 K0C, K73 K1C, K74 K2C, K75 K3C, K76 K4C, K77 K4C, K78 K0D, K79 K0D, K8 K40, K80 K1D, K81 K2D, K82 K2D, K83 K3D, K84 K3C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

Commit message: - FIxed bug in wiring (missing connections)
Connections:
- net Col8: now also K50.1
- net at K50.2: now also D40.2 (A)
Changed lines of the file:
@@
 Wire Notes Line
 	500  500  10950 500
+Wire Wire Line
+	6850 600  6850 850
+Wire Wire Line
+	6250 850  6250 1150
 $EndSCHEMATC

Commit message: - First draw for Rev. B
Parts:
- DK0: renamed from D1; value D -> D00
- DK1: renamed from D2; value D -> D10
- DK10: renamed from D6; value D -> D01
- DK11: renamed from D7; value D -> D11
- DK12: renamed from D8; value D -> D21
- DK13: renamed from D9; value D -> D31
- DK14: renamed from D10; value D -> D41
- DK2: renamed from D3; value D -> D20
- DK20: renamed from D11; value D -> D02
- DK21: renamed from D12; value D -> D12
- DK22: renamed from D13; value D -> D22
- DK23: renamed from D14; value D -> D32
- DK24: renamed from D15; value D -> D42
- DK3: renamed from D4; value D -> D30
- DK30: renamed from D16; value D -> D03
- DK31: renamed from D17; value D -> D13
- DK32: renamed from D18; value D -> D23
- DK33: renamed from D19; value D -> D33
- DK4: renamed from D5; value D -> D40
- DK40: renamed from D21; value D -> D04
- DK41: renamed from D22; value D -> D14
- DK42: renamed from D23; value D -> D24
- DK43: renamed from D24; value D -> D34
- DK50: renamed from D26; value D -> D05
- DK51: renamed from D27; value D -> D15
- DK52: renamed from D28; value D -> D25
- DK53: renamed from D29; value D -> D35
- DK6: renamed from D31; value D -> D60
- DK61: renamed from D32; value D -> D16
- DK62: renamed from D33; value D -> D26
- DK63: renamed from D34; value D -> D36
- DK64: renamed from D35; value D -> D46
- DK70: renamed from D36; value D -> D07
- DK71: renamed from D37; value D -> D17
- DK72: renamed from D38; value D -> D27
- DK73: renamed from D39; value D -> D37
- DK80: renamed from D40; value D -> D08
- DK81: renamed from D41; value D -> D18
- DK82: renamed from D42; value D -> D28
- DK83: renamed from D43; value D -> D38
- DK90: renamed from D44; value D -> D09
- DK91: renamed from D45; value D -> D19
- DK92: renamed from D46; value D -> D29
- DK93: renamed from D47; value D -> D39
- DK94: renamed from D48; value D -> D49
- DKA0: renamed from D49; value D -> D0A
- DKA1: renamed from D50; value D -> DA1
- DKA2: renamed from D51; value D -> D2A
- DKA3: renamed from D52; value D -> D3A
- DKA4: renamed from D53; value D -> D4A
- DKB0: renamed from D54; value D -> D0B
- DKB1: renamed from D55; value D -> D1B
- DKB2: renamed from D56; value D -> D2B
- DKB3: renamed from D57; value D -> D3B
- DKB4: renamed from D58; value D -> D4B
- DKC1: renamed from D60; value D -> D1C
- DKC2: renamed from D61; value D -> D2C
- DKC3: renamed from D62; value D -> D3C
- DKC4: renamed from D63; value D -> D4C
- DKD0: renamed from D64; value D -> DKD0
- DKD1: renamed from D65; value D -> D1D
- DKD2: renamed from D66; value D -> D2D
- DKD3: renamed from D67; value D -> D3D
- DKD4: renamed from D68; value D -> D4D
- KDC0: renamed from D59; value D -> D0C
- renumbered K1 to K0, K2 to K10, K9 to K100, K10 to K110, K11 to K120, K12 to K130, K13 to K140, K14 to K141, K3 to K20, K15 to K200, K4 to K21, K16 to K210, K17 to K220, K18 to K230, K19 to K240, K20 to K241, K5 to K30, K21 to K300, K6 to K31, K22 to K310, K23 to K320, K24 to K330, K7 to K40, K27 to K400, K8 to K41, K28 to K410, K29 to K420, K30 to K430, K77 to K4C1, K32 to K500, K33 to K510, K34 to K520, K35 to K530, K38 to K600, K39 to K610, K40 to K620, K41 to K630, K42 to K640, K44 to K641, K45 to K642, K46 to K700, K47 to K710, K48 to K720, K49 to K730, K50 to K800, K51 to K810, K52 to K820, K53 to K830, K54 to K900, K55 to K910, K56 to K920, K57 to K930, K58 to K940, K59 to KA0, K60 to KA10, K61 to KA20, K62 to KA30, K63 to KA40, K64 to KA41, K65 to KB0, K66 to KB10, K67 to KB20, K68 to KB30, K69 to KB40, K70 to KB41, K71 to KB42, K72 to KC0, K73 to KC10, K74 to KC20, K75 to KC30, K31 to KC31, K84 to KC32, K76 to KC40, K78 to KD0, K79 to KD1, K80 to KD10, K25 to KD20, K81 to KD21, K82 to KD22, K83 to KD30, K26 to KD31, K85 to KD40, K86 to KD41
Connections:
- net Col0: now also DK0.2 (A), DK1.2 (A), DK2.2 (A), DK3.2 (A), DK4.2 (A); no longer K0.1, K10.1, K20.1, K21.2, K30.1, K31.1, K40.1, K41.1
- net Col1: now also DK10.2 (A), DK11.2 (A), DK12.2 (A), DK13.2 (A), DK14.2 (A); no longer K100.1, K110.1, K120.1, K130.1, K140.1, K141.1
- net Col2: now also DK20.2 (A), DK21.2 (A), DK22.2 (A), DK23.2 (A), DK24.2 (A); no longer K200.1, K210.1, K220.1, K230.1, K240.1, K241.1
- net Col3: now also DK30.2 (A), DK31.2 (A), DK32.2 (A), DK33.2 (A); no longer K300.1, K310.1, K320.1, K330.1
- net Col4: now also DK40.2 (A), DK41.2 (A), DK42.2 (A), DK43.2 (A); no longer K400.1, K410.1, K420.1, K430.1
- net Col5: now also DK50.2 (A), DK51.2 (A), DK52.2 (A), DK53.2 (A); no longer K500.1, K510.1, K520.1, K530.1
- net Col6: now also DK6.2 (A), DK61.2 (A), DK62.2 (A), DK63.2 (A), DK64.2 (A); no longer K600.1, K610.1, K620.1, K630.1, K640.1, K641.1, K642.2
- net Col7: now also DK70.2 (A), DK71.2 (A), DK72.2 (A), DK73.2 (A); no longer K700.1, K710.1, K720.1, K730.1
- net Col8: now also DK80.2 (A), DK81.2 (A), DK82.2 (A), DK83.2 (A); no longer K800.1, K810.1, K820.1, K830.1
- net Col9: now also DK90.2 (A), DK91.2 (A), DK92.2 (A), DK93.2 (A), DK94.2 (A); no longer K900.1, K910.1, K920.1, K930.1, K940.1
- net ColA: now also DKA0.2 (A), DKA1.2 (A), DKA2.2 (A), DKA3.2 (A), DKA4.2 (A); no longer KA0.1, KA10.1, KA20.1, KA30.1, KA40.1, KA41.1
- net ColB: now also DKB0.2 (A), DKB1.2 (A), DKB2.2 (A), DKB3.2 (A), DKB4.2 (A); no longer KB0.1, KB10.1, KB20.1, KB30.1, KB40.1, KB41.1, KB42.1
- net ColC: now also DKC1.2 (A), DKC2.2 (A), DKC3.2 (A), DKC4.2 (A), KDC0.2 (A); no longer K4C1.1, KC0.1, KC10.1, KC20.1, KC30.1, KC31.2, KC32.1, KC40.1
- net ColD: now also DKD0.2 (A), DKD1.2 (A), DKD2.2 (A), DKD3.2 (A), DKD4.2 (A); no longer KD0.1, KD1.1, KD10.1, KD20.1, KD21.1, KD22.1, KD30.1, KD31.2, KD40.1, KD41.1
- net Row0: now also K0.2, K100.2, K200.2, K300.2, K400.2, K500.2, K600.2, K700.2, K800.2, K900.2, KA0.2, KB0.2, KC0.2, KD0.2, KD1.2; no longer DK0.1 (K), DK10.1 (K), DK20.1 (K), DK30.1 (K), DK40.1 (K), DK50.1 (K), DK6.1 (K), DK70.1 (K), DK80.1 (K), DK90.1 (K), DKA0.1 (K), DKB0.1 (K), DKD0.1 (K), KDC0.1 (K)
- net Row1: now also K10.2, K110.2, K210.2, K310.2, K410.2, K510.2, K610.2, K710.2, K810.2, K910.2, KA10.2, KB10.2, KC10.2, KD10.2; no longer DK1.1 (K), DK11.1 (K), DK21.1 (K), DK31.1 (K), DK41.1 (K), DK51.1 (K), DK61.1 (K), DK71.1 (K), DK81.1 (K), DK91.1 (K), DKA1.1 (K), DKB1.1 (K), DKC1.1 (K), DKD1.1 (K)
- net Row2: now also K120.2, K20.2, K21.2, K220.2, K320.2, K420.2, K520.2, K620.2, K720.2, K820.2, K920.2, KA20.2, KB20.2, KC20.2, KD20.2, KD21.2, KD22.2; no longer DK12.1 (K), DK2.1 (K), DK22.1 (K), DK32.1 (K), DK42.1 (K), DK52.1 (K), DK62.1 (K), DK72.1 (K), DK82.1 (K), DK92.1 (K), DKA2.1 (K), DKB2.1 (K), DKC2.1 (K), DKD2.1 (K)
- net Row3: now also K130.2, K230.2, K30.2, K31.2, K330.2, K430.2, K530.2, K630.2, K730.2, K830.2, K930.2, KA30.2, KB30.2, KC30.2, KC31.2, KC32.2, KD30.2, KD31.2; no longer DK13.1 (K), DK23.1 (K), DK3.1 (K), DK33.1 (K), DK43.1 (K), DK53.1 (K), DK63.1 (K), DK73.1 (K), DK83.1 (K), DK93.1 (K), DKA3.1 (K), DKB3.1 (K), DKC3.1 (K), DKD3.1 (K)
- net Row4: now also K140.2, K141.2, K240.2, K241.2, K40.2, K41.2, K4C1.2, K640.2, K641.1, K642.2, K940.2, KA40.2, KA41.2, KB40.2, KB41.2, KB42.2, KC40.2, KD40.2, KD41.2; no longer DK14.1 (K), DK24.1 (K), DK4.1 (K), DK64.1 (K), DK94.1 (K), DKA4.1 (K), DKB4.1 (K), DKC4.1 (K), DKD4.1 (K)
- net at K641.2, K642.1: now also DK64.1 (K), K640.1; no longer DK64.2 (A), K640.2
- new net: DK0.1 (K), K0.1
- new net: DK10.1 (K), K100.1
- new net: DK20.1 (K), K200.1
- new net: DK30.1 (K), K300.1
- new net: DK40.1 (K), K400.1
- new net: DK50.1 (K), K500.1
- new net: DK6.1 (K), K600.1
- new net: DK70.1 (K), K700.1
- new net: DK80.1 (K), K800.1
- new net: DK90.1 (K), K900.1
- new net: DKA0.1 (K), KA0.1
- new net: DKB0.1 (K), KB0.1
- new net: KC0.1, KDC0.1 (K)
- new net: DKD0.1 (K), KD0.1, KD1.1
- new net: DK1.1 (K), K10.1
- new net: DK11.1 (K), K110.1
- new net: DK21.1 (K), K210.1
- new net: DK31.1 (K), K310.1
- new net: DK41.1 (K), K410.1
- new net: DK51.1 (K), K510.1
- new net: DK61.1 (K), K610.1
- new net: DK71.1 (K), K710.1
- new net: DK81.1 (K), K810.1
- new net: DK91.1 (K), K910.1
- new net: DKA1.1 (K), KA10.1
- new net: DKB1.1 (K), KB10.1
- new net: DKC1.1 (K), KC10.1
- new net: DKD1.1 (K), KD10.1
- new net: DK2.1 (K), K20.1, K21.1
- new net: DK12.1 (K), K120.1
- new net: DK22.1 (K), K220.1
- new net: DK32.1 (K), K320.1
- new net: DK42.1 (K), K420.1
- new net: DK52.1 (K), K520.1
- new net: DK62.1 (K), K620.1
- new net: DK72.1 (K), K720.1
- new net: DK82.1 (K), K820.1
- new net: DK92.1 (K), K920.1
- new net: DKA2.1 (K), KA20.1
- new net: DKB2.1 (K), KB20.1
- new net: DKC2.1 (K), KC20.1
- new net: DKD2.1 (K), KD20.1, KD21.1, KD22.1
- new net: DKD3.1 (K), KD30.1, KD31.1
- new net: DKC3.1 (K), KC30.1, KC31.1, KC32.1
- new net: DK3.1 (K), K30.1, K31.1
- new net: DK13.1 (K), K130.1
- new net: DK23.1 (K), K230.1
- new net: DK33.1 (K), K330.1
- new net: DK43.1 (K), K430.1
- new net: DK53.1 (K), K530.1
- new net: DK63.1 (K), K630.1
- new net: DK73.1 (K), K730.1
- new net: DK83.1 (K), K830.1
- new net: DK93.1 (K), K930.1
- new net: DKA3.1 (K), KA30.1
- new net: DKB3.1 (K), KB30.1
- new net: DK4.1 (K), K40.1, K41.1
- new net: DK14.1 (K), K140.1, K141.1
- new net: DK24.1 (K), K240.1, K241.1
- new net: DK94.1 (K), K940.1
- new net: DKA4.1 (K), KA40.1, KA41.1
- new net: DKB4.1 (K), KB40.1, KB41.1, KB42.1
- new net: DKC4.1 (K), K4C1.1, KC40.1
- new net: DKD4.1 (K), KD40.1, KD41.1

Commit message: - Simplifying routing (2/n) + fixed bug for RShift
Connections:
- net Row3: now also KD30.1; no longer KD30.2
- net at DKD3.1 (K), KD31.1: now also KD30.2; no longer KD30.1
Changed lines of the file:
@@
 F 3 "" H 10050 4200 60  0000 C CNN
 	1    10050 4200
-	1    0    0    -1
+	-1   0    0    1
 $EndComp
 $Comp

Commit message: - First commit for splitted spacebar
Parts:
- added DK54: D45, Footprint:D_SOD123, symbol D
- added DK74: D47, Footprint:D_SOD123, symbol D
- added K540: K465, Footprint:Mx_275, symbol KEYSW
- added K643: K46, Footprint:Mx_100, symbol KEYSW
- added K740: K47, Footprint:Mx_225, symbol KEYSW
Connections:
- net Col5: now also DK54.2 (A)
- net Col7: now also DK74.2 (A)
- net Row4: now also K540.2, K643.1, K740.2
- net at DK64.1 (K), K640.1, K641.2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: now also K643.2
- new net: DK54.1 (K), K540.1
- new net: DK74.1 (K), K740.1
Changed lines of the file:
@@
 Connection ~ 9050 5850
 Connection ~ 9750 5850
+$Comp
+L KEYSW K540
+U 1 1 59DE9804
+P 4450 5550
+F 0 "K540" H 4400 5550 60  0001 C CNN
+F 1 "K465" H 4450 5450 60  0000 C CNN
+F 2 "Footprint:Mx_275" H 4450 5550 60  0001 C CNN
+F 3 "" H 4450 5550 60  0000 C CNN
+	1    4450 5550
+	1    0    0    -1
+$EndComp
+$Comp
+L KEYSW K740
+U 1 1 59DE980F
+P 5850 5550
+F 0 "K740" H 5800 5550 60  0001 C CNN
+F 1 "K47" H 5850 5450 60  0000 C CNN
+F 2 "Footprint:Mx_225" H 5850 5550 60  0001 C CNN
+F 3 "" H 5850 5550 60  0000 C CNN
+	1    5850 5550
+	1    0    0    -1
+$EndComp
+Text GLabel 4750 5250 0    60   Input ~ 0
+Col5
+Text GLabel 6150 5250 0    60   Input ~ 0
+Col7
+$Comp
+L D DK74
+U 1 1 59DE981E
+P 6150 5400
+F 0 "DK74" H 6150 5500 50  0001 C CNN
+F 1 "D47" H 6150 5300 50  0001 C CNN
+F 2 "Footprint:D_SOD123" H 6150 5400 50  0001 C CNN
+F 3 "" H 6150 5400 50  0000 C CNN
+	1    6150 5400
+	0    -1   -1   0
+$EndComp
+$Comp
+L D DK54
+U 1 1 59DE9829
+P 4750 5400
+F 0 "DK54" H 4750 5500 50  0001 C CNN
+F 1 "D45" H 4750 5300 50  0001 C CNN
+F 2 "Footprint:D_SOD123" H 4750 5400 50  0001 C CNN
+F 3 "" H 4750 5400 50  0000 C CNN
+	1    4750 5400
+	0    -1   -1   0
+$EndComp
+$Comp
+L KEYSW K643
+U 1 1 59DE985B
+P 5150 5700
+F 0 "K643" H 5100 5700 60  0001 C CNN
+F 1 "K46" H 5150 5600 60  0001 C CNN
+F 2 "Footprint:Mx_100" H 5150 5700 60  0001 C CNN
+F 3 "" H 5150 5700 60  0000 C CNN
+	1    5150 5700
+	-1   0    0    1
+$EndComp
+Wire Wire Line
+	4150 5550 4150 6400
+Connection ~ 4150 6400
+Wire Wire Line
+	5550 5550 5550 6400
+Connection ~ 5550 6400
+Connection ~ 4850 5700
+Connection ~ 5450 5700
 $EndSCHEMATC

Commit message: - Added Splitted spacebar
Connections:
- net Row4: now also K642.1, K643.2; no longer K642.2, K643.1
- net at DK64.1 (K), K640.1, K641.2: now also K642.2, K643.1; no longer K642.1, K643.2
Changed lines of the file:
@@
 F 3 "" H 5150 6150 60  0000 C CNN
 	1    5150 6150
-	1    0    0    -1
+	-1   0    0    1
 $EndComp
 $Comp
@@
 F 3 "" H 5150 5700 60  0000 C CNN
 	1    5150 5700
-	-1   0    0    1
-$EndComp
-Wire Wire Line
+	1    0    0    -1
+$EndComp
+Wire Wire Line

Commit message: - Routing and moved components near holes
Parts:
- K540: value K465 -> K45
Changed lines of the file:
@@
 P 4450 5550
 F 0 "K540" H 4400 5550 60  0001 C CNN
-F 1 "K465" H 4450 5450 60  0000 C CNN
+F 1 "K45" H 4450 5450 60  0000 C CNN
 F 2 "Footprint:Mx_275" H 4450 5550 60  0001 C CNN
 F 3 "" H 4450 5550 60  0000 C CNN
