File: Kicad/MATRIX.sch (KiCad schematic (older format))
At the start: 153 parts, among them K0 K00, K10 K10, K100 K01, K110 K11, K120 K21, K130 K31, K140 K41, K141 K41, K20 K20, K200 K02, K21 K20, K210 K12, K220 K22, K230 K32, K240 K42, K241 K42, K30 K30, K300 K03, K31 K30, K310 K13, K320 K23, K330 K33, K40 K40, K400 K04, K41 K40, K410 K14, K420 K24, K430 K34, K4C1 K4C, K500 K05, K510 K15, K520 K25, K530 K35, K540 K45, K600 K06, K610 K16, K620 K26, K630 K36, K640 K46, K641 K46, K642 K46, K643 K46, K700 K07, K710 K17, K720 K27, K730 K37, K740 K47, K800 K08, K810 K18, K820 K28, K830 K38, K900 K09, K910 K19, K920 K29, K930 K39, K940 K49

Commit message: Removed useless libraries
Merging all components in one library file to simplify maintenance
Parts:
- K0, K10, K100, K110, K120, K130, K140, K141, K20, K200, K21, K210, K220, K230, K240, K241, K30, K300, K31, K310, K320, K330, K40, K400, K41, K410, K420, K430, K4C1, K500, K510, K520, K530, K540, K600, K610, K620, K630, K640, K641, K642, K643, K700, K710, K720, K730, K740, K800, K810, K820, K830, K900, K910, K920, K930, K940, KA0, KA10, KA20, KA30, KA40, KA41, KB0, KB10, KB20, KB30, KB40, KB41, KB42, KC0, KC10, KC20, KC30, KC31, KC32, KC40, KD0, KD1, KD10, KD20, KD21, KD22, KD30, KD31, KD40, KD41: manf# (none) -> MX1A-C1NW
Connections:
- no-connect marks 0 -> 1
