File: Kicad/MATRIX.sch (KiCad schematic (older format))
At the start: 153 parts, among them K0 K00, K10 K10, K100 K01, K110 K11, K120 K21, K130 K31, K140 K41, K141 K41, K20 K20, K200 K02, K21 K20, K210 K12, K220 K22, K230 K32, K240 K42, K241 K42, K30 K30, K300 K03, K31 K30, K310 K13, K320 K23, K330 K33, K40 K40, K400 K04, K41 K40, K410 K14, K420 K24, K430 K34, K4C1 K4C, K500 K05, K510 K15, K520 K25, K530 K35, K540 K45, K600 K06, K610 K16, K620 K26, K630 K36, K640 K46, K641 K46, K642 K46, K643 K46, K700 K07, K710 K17, K720 K27, K730 K37, K740 K47, K800 K08, K810 K18, K820 K28, K830 K38, K900 K09, K910 K19, K920 K29, K930 K39, K940 K49

Commit message: - Added ivan ivanovitch layout
Parts:
- added K142: K41, Footprint:Mx_150, symbol KEYSW
Connections:
- net Row4: now also K142.1
- net at DK14.1 (K), K140.1, K141.1: now also K142.2
Changed lines of the file:
@@
 EESchema Schematic File Version 2
 LIBS:kicad_parts
-LIBS:DK60TP-cache
 EELAYER 25 0
 EELAYER END
@@
 	2050 5550 2050 6400
 Wire Wire Line
-	1950 5550 1950 5850
+	1950 5550 1950 6150
 Wire Wire Line
 	1350 5550 1350 6400
@@
 Connection ~ 5450 5700
 NoConn ~ -200 1000
+$Comp
+L KEYSW K142
+U 1 1 59EC7A8F
+P 1650 6150
+F 0 "K142" H 1600 6150 60  0001 C CNN
+F 1 "K41" H 1650 6050 60  0001 C CNN
+F 2 "Footprint:Mx_150" H 1650 6150 60  0001 C CNN
+F 3 "https://search.kemet.com/component-edge/download/datasheet/C0805C220J5GACTU.pdf" H 1650 6150 60  0001 C CNN
+F 4 "MX1A-C1NW" H 1650 1200 60  0001 C CNN "manf#"
+	1    1650 6150
+	-1   0    0    1
+$EndComp
+Connection ~ 1950 5850
+Connection ~ 1350 6150
 $EndSCHEMATC
