File: Kicad/BACKLIT.sch (KiCad schematic (older format))
At the start: 88 parts, among them U1 PAM2804

Commit message: - First draw for Rev. B
Parts:
- renumbered D20 to BL0, D25 to BL10, D71 to BL100, D72 to BL110, D73 to BL120, D74 to BL130, D80 to BL140, D85 to BL141, D30 to BL20, D76 to BL200, D137 to BL21, D77 to BL210, D78 to BL220, D79 to BL230, D90 to BL240, D95 to BL241, D69 to BL30, D81 to BL300, D148 to BL31, D82 to BL310, D83 to BL320, D84 to BL330, D70 to BL40, D86 to BL400, D75 to BL41, D87 to BL410, D88 to BL420, D89 to BL430, D91 to BL500, D92 to BL510, D93 to BL520, D94 to BL530, D96 to BL600, D97 to BL610, D98 to BL620, D99 to BL630, D100 to BL640, D105 to BL641, D110 to BL642, D101 to BL700, D102 to BL710, D103 to BL720, D104 to BL750, D106 to BL800, D107 to BL810, D108 to BL820, D109 to BL830, D111 to BL900, D112 to BL910, D113 to BL920, D114 to BL930, D141 to BL940, D116 to BLA0, D117 to BLA10, D118 to BLA20, D119 to BLA30, D115 to BLA40, D120 to BLA41, D121 to BLB0, D122 to BLB10, D123 to BLB20, D124 to BLB30, D125 to BLB40, D130 to BLB41, D135 to BLB42, D126 to BLC0, D127 to BLC10, D128 to BLC20, D129 to BLC30, D134 to BLC31, D139 to BLC32, D140 to BLC40, D143 to BLC41, D131 to BLD0, D136 to BLD1, D132 to BLD10, D133 to BLD20, D138 to BLD21, D146 to BLD22, D142 to BLD30, D145 to BLD31, D144 to BLD40, D147 to BLD41
Other:
- moved on the sheet: BL0, BL10, BL100, BL110, BL120, BL130, BL140, BL141, BL20, BL200, BL21, BL210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

Commit message: - Routing and moved components near holes
Parts:
- added BL540, BL740: LED, Footprint:LED_TH_BIVAR, symbol LED
Connections:
- net LED_AN: now also BL540.2 (A), BL740.2 (A)
- net LED_CATH: now also BL540.1 (K), BL740.1 (K)
Other:
- moved on the sheet: BL640, BL641, BL642, BLA40, BLA41, BLB40, BLB41, BLB42, BLC40, BLC41, BLD40, BLD41
Changed lines of the file:
@@
 L LED BL640
 U 1 1 59332BFB
-P 3650 5700
-F 0 "BL640" H 3650 5800 50  0000 C CNN
-F 1 "LED" H 3650 5600 50  0001 C CNN
-F 2 "Footprint:LED_TH_BIVAR" H 3650 5700 50  0001 C CNN
-F 3 "" H 3650 5700 50  0000 C CNN
-	1    3650 5700
-	0    -1   -1   0
-$EndComp
-$Comp
-L LED BL641
-U 1 1 59332C01
 P 3950 5700
-F 0 "BL641" H 3950 5800 50  0000 C CNN
+F 0 "BL640" H 3950 5800 50  0000 C CNN
 F 1 "LED" H 3950 5600 50  0001 C CNN
 F 2 "Footprint:LED_TH_BIVAR" H 3950 5700 50  0001 C CNN
@@
 $EndComp
 $Comp
-L LED BL642
-U 1 1 59332C07
+L LED BL641
+U 1 1 59332C01
 P 4250 5700
-F 0 "BL642" H 4250 5800 50  0000 C CNN
+F 0 "BL641" H 4250 5800 50  0000 C CNN
 F 1 "LED" H 4250 5600 50  0001 C CNN
 F 2 "Footprint:LED_TH_BIVAR" H 4250 5700 50  0001 C CNN
@@
 $EndComp
 $Comp
-L LED BLA40
-U 1 1 59332C0D
+L LED BL642
+U 1 1 59332C07
 P 4550 5700
-F 0 "BLA40" H 4550 5800 50  0000 C CNN
+F 0 "BL642" H 4550 5800 50  0000 C CNN
 F 1 "LED" H 4550 5600 50  0001 C CNN
 F 2 "Footprint:LED_TH_BIVAR" H 4550 5700 50  0001 C CNN
@@
 $EndComp
 $Comp
-L LED BLA41
-U 1 1 59332C13
-P 4850 5700
-F 0 "BLA41" H 4850 5800 50  0000 C CNN
-F 1 "LED" H 4850 5600 50  0001 C CNN
-F 2 "Footprint:LED_TH_BIVAR" H 4850 5700 50  0001 C CNN
-F 3 "" H 4850 5700 50  0000 C CNN
-	1    4850 5700
-	0    -1   -1   0
-$EndComp
-$Comp
-L LED BLB40
-U 1 1 59332C19
+L LED BLA40
+U 1 1 59332C0D
 P 5150 5700
-F 0 "BLB40" H 5150 5800 50  0000 C CNN
+F 0 "BLA40" H 5150 5800 50  0000 C CNN
 F 1 "LED" H 5150 5600 50  0001 C CNN
 F 2 "Footprint:LED_TH_BIVAR" H 5150 5700 50  0001 C CNN
@@
 $EndComp
 $Comp
-L LED BLB41
-U 1 1 59332C1F
+L LED BLA41
+U 1 1 59332C13
 P 5450 5700
-F 0 "BLB41" H 5450 5800 50  0000 C CNN
+F 0 "BLA41" H 5450 5800 50  0000 C CNN
 F 1 "LED" H 5450 5600 50  0001 C CNN
 F 2 "Footprint:LED_TH_BIVAR" H 5450 5700 50  0001 C CNN
@@
 $EndComp
 $Comp
-L LED BLB42
-U 1 1 59332C25
+L LED BLB40
+U 1 1 59332C19
 P 5750 5700
-F 0 "BLB42" H 5750 5800 50  0000 C CNN
+F 0 "BLB40" H 5750 5800 50  0000 C CNN
 F 1 "LED" H 5750 5600 50  0001 C CNN
 F 2 "Footprint:LED_TH_BIVAR" H 5750 5700 50  0001 C CNN
@@
 $EndComp
 $Comp
-L LED BLC40
-U 1 1 59332C2B
+L LED BLB41
+U 1 1 59332C1F
 P 6050 5700
-F 0 "BLC40" H 6050 5800 50  0000 C CNN
+F 0 "BLB41" H 6050 5800 50  0000 C CNN
 F 1 "LED" H 6050 5600 50  0001 C CNN
 F 2 "Footprint:LED_TH_BIVAR" H 6050 5700 50  0001 C CNN
@@
 $EndComp
 $Comp
-L LED BLC41
-U 1 1 59332C31
+L LED BLB42
+U 1 1 59332C25
 P 6350 5700
-F 0 "BLC41" H 6350 5800 50  0000 C CNN
+F 0 "BLB42" H 6350 5800 50  0000 C CNN
 F 1 "LED" H 6350 5600 50  0001 C CNN
 F 2 "Footprint:LED_TH_BIVAR" H 6350 5700 50  0001 C CNN
@@
 	0    -1   -1   0
 $EndComp
-Text GLabel 1650 5900 0    60   Input ~ 0
-LED_CATH
-$Comp
-L LED BLD40
-U 1 1 59332EAD
+$Comp
+L LED BLC40
+U 1 1 59332C2B
 P 6650 5700
-F 0 "BLD40" H 6650 5800 50  0000 C CNN
+F 0 "BLC40" H 6650 5800 50  0000 C CNN
 F 1 "LED" H 6650 5600 50  0001 C CNN
 F 2 "Footprint:LED_TH_BIVAR" H 6650 5700 50  0001 C CNN
 F 3 "" H 6650 5700 50  0000 C CNN
 	1    6650 5700
+	0    -1   -1   0
+$EndComp
+$Comp
+L LED BLC41
+U 1 1 59332C31
+P 6950 5700
+F 0 "BLC41" H 6950 5800 50  0000 C CNN
+F 1 "LED" H 6950 5600 50  0001 C CNN
+F 2 "Footprint:LED_TH_BIVAR" H 6950 5700 50  0001 C CNN
+F 3 "" H 6950 5700 50  0000 C CNN
+	1    6950 5700
+	0    -1   -1   0
+$EndComp
+Text GLabel 1650 5900 0    60   Input ~ 0
+LED_CATH
+$Comp
+L LED BLD40
+U 1 1 59332EAD
+P 7250 5700
+F 0 "BLD40" H 7250 5800 50  0000 C CNN
+F 1 "LED" H 7250 5600 50  0001 C CNN
+F 2 "Footprint:LED_TH_BIVAR" H 7250 5700 50  0001 C CNN
+F 3 "" H 7250 5700 50  0000 C CNN
+	1    7250 5700
 	0    -1   -1   0
 $EndComp
@@
 L LED BLD41
 U 1 1 5934C32E
-P 6950 5700
-F 0 "BLD41" H 6950 5800 50  0000 C CNN
-F 1 "LED" H 6950 5600 50  0001 C CNN
-F 2 "Footprint:LED_TH_BIVAR" H 6950 5700 50  0001 C CNN
-F 3 "" H 6950 5700 50  0000 C CNN
-	1    6950 5700
+P 7550 5700
+F 0 "BLD41" H 7550 5800 50  0000 C CNN
+F 1 "LED" H 7550 5600 50  0001 C CNN
+F 2 "Footprint:LED_TH_BIVAR" H 7550 5700 50  0001 C CNN
+F 3 "" H 7550 5700 50  0000 C CNN
+	1    7550 5700
 	0    -1   -1   0
 $EndComp
@@
 Connection ~ 3050 5550
 Connection ~ 3350 5550
-Connection ~ 3650 5550
 Connection ~ 3950 5550
 Connection ~ 4250 5550
 Connection ~ 4550 5550
-Connection ~ 4850 5550
 Connection ~ 5150 5550
 Connection ~ 5450 5550
 Connection ~ 5750 5550
 Connection ~ 6050 5550
-Wire Wire Line
-	6350 5900 6350 5850
+Connection ~ 6350 5550
+Connection ~ 6650 5550
+Wire Wire Line
+	6950 5900 6950 5850
+Wire Wire Line
+	6650 5850 6650 5900
+Connection ~ 6650 5900
+Wire Wire Line
+	6350 5850 6350 5900
+Connection ~ 6350 5900
 Wire Wire Line
 	6050 5850 6050 5900
@@
 Connection ~ 5150 5900
 Wire Wire Line
-	4850 5850 4850 5900
-Connection ~ 4850 5900
-Wire Wire Line
 	4550 5850 4550 5900
 Connection ~ 4550 5900
@@
 Connection ~ 3950 5900
 Wire Wire Line
-	3650 5850 3650 5900
-Connection ~ 3650 5900
-Wire Wire Line
 	3350 5850 3350 5900
 Connection ~ 3350 5900
@@
 	1850 5850 1850 5900
 Connection ~ 1850 5900
-Connection ~ 6350 5550
-Wire Wire Line
-	6650 5900 6650 5850
-Connection ~ 6350 5900
+Connection ~ 6950 5550
+Wire Wire Line
+	7250 5900 7250 5850
+Connection ~ 6950 5900
 Connection ~ 6350 4900
 Connection ~ 6350 5250
@@
 	6650 5250 6650 5200
 Wire Wire Line
-	1650 5550 6950 5550
-Wire Wire Line
-	1650 5900 6950 5900
+	1650 5550 7550 5550
+Wire Wire Line
+	1650 5900 7550 5900
 Wire Wire Line
 	3000 1750 2050 1750
@@
 Wire Wire Line
 	5750 3950 1650 3950
-Connection ~ 6650 5550
-Wire Wire Line
-	6950 5900 6950 5850
-Connection ~ 6650 5900
-Wire Notes Line
-	900  2650 7250 2650
-Wire Notes Line
-	7250 2650 7250 6200
-Wire Notes Line
-	7250 6200 900  6200
+Connection ~ 7250 5550
+Wire Wire Line
+	7550 5900 7550 5850
+Connection ~ 7250 5900
+Wire Notes Line
+	900  2650 7900 2650
+Wire Notes Line
+	7900 2650 7900 6200
+Wire Notes Line
+	7900 6200 900  6200
 Wire Notes Line
 	900  6200 900  2650
+$Comp
+L LED BL540
+U 1 1 59E13C04
+P 3650 5700
+F 0 "BL540" H 3650 5800 50  0000 C CNN
+F 1 "LED" H 3650 5600 50  0001 C CNN
+F 2 "Footprint:LED_TH_BIVAR" H 3650 5700 50  0001 C CNN
+F 3 "" H 3650 5700 50  0000 C CNN
+	1    3650 5700
+	0    -1   -1   0
+$EndComp
+Connection ~ 3650 5550
+Wire Wire Line
+	3650 5850 3650 5900
+Connection ~ 3650 5900
+$Comp
+L LED BL740
+U 1 1 59E1B57C
+P 4850 5700
+F 0 "BL740" H 4850 5800 50  0000 C CNN
+F 1 "LED" H 4850 5600 50  0001 C CNN
+F 2 "Footprint:LED_TH_BIVAR" H 4850 5700 50  0001 C CNN
+F 3 "" H 4850 5700 50  0000 C CNN
+	1    4850 5700
+	0    -1   -1   0
+$EndComp
+Wire Wire Line
+	4850 5850 4850 5900
+Connection ~ 4850 5900
+Connection ~ 4850 5550
 $EndSCHEMATC

Commit message: Removed useless libraries
Merging all components in one library file to simplify maintenance
Parts:
- C10, C11: manf# (none) -> CC0805ZKY5V7BB106
- L1: manf# (none) -> 744766904
- R5: manf# (none) -> RL0805FR-7W0R5L
- U1: manf# (none) -> PAM2804AAB010
Changed lines of the file:
@@
 EESchema Schematic File Version 2
-LIBS:74xgxx
-LIBS:74xx
-LIBS:ac-dc
-LIBS:actel
-LIBS:adc-dac
-LIBS:allegro
-LIBS:Altera
-LIBS:analog_devices
-LIBS:analog_switches
-LIBS:audio
-LIBS:battery_management
-LIBS:bbd
-LIBS:bosch
-LIBS:brooktre
-LIBS:cmos4000
-LIBS:cmos_ieee
-LIBS:conn
-LIBS:contrib
-LIBS:cypress
-LIBS:dc-dc
-LIBS:device
-LIBS:digital-audio
-LIBS:diode
-LIBS:display
-LIBS:dsp
-LIBS:elec-unifil
-LIBS:ESD_Protection
-LIBS:ftdi
-LIBS:gennum
-LIBS:graphic_symbols
-LIBS:hc11
-LIBS:infineon
-LIBS:intel
-LIBS:interface
-LIBS:intersil
-LIBS:ir
-LIBS:Lattice
-LIBS:leds
-LIBS:LEM
-LIBS:linear
-LIBS:logic_programmable
-LIBS:maxim
-LIBS:mechanical
-LIBS:memory
-LIBS:microchip
-LIBS:microchip_dspic33dsc
-LIBS:microchip_pic10mcu
-LIBS:microchip_pic12mcu
-LIBS:microchip_pic16mcu
-LIBS:microchip_pic18mcu
-LIBS:microchip_pic24mcu
-LIBS:microchip_pic32mcu
-LIBS:microcontrollers
-LIBS:modules
-LIBS:motor_drivers
-LIBS:motorola
-LIBS:motors
-LIBS:msp430
-LIBS:nordicsemi
-LIBS:nxp
-LIBS:nxp_armmcu
-LIBS:onsemi
-LIBS:opto
-LIBS:Oscillators
-LIBS:philips
-LIBS:power
-LIBS:powerint
-LIBS:Power_Management
-LIBS:pspice
-LIBS:references
-LIBS:regul
-LIBS:relays
-LIBS:rfcom
-LIBS:RFSolutions
-LIBS:sensors
-LIBS:silabs
-LIBS:siliconi
-LIBS:stm8
-LIBS:stm32
-LIBS:supertex
-LIBS:switches
-LIBS:texas
-LIBS:transf
-LIBS:transistors
-LIBS:triac_thyristor
-LIBS:ttl_ieee
-LIBS:valves
-LIBS:video
-LIBS:wiznet
-LIBS:Xicor
-LIBS:xilinx
-LIBS:zetex
-LIBS:Zilog
 LIBS:keyboard_parts
-LIBS:mkl27z256vfm4
-LIBS:Trackpad
-LIBS:TS65
 LIBS:DK60TP-cache
 EELAYER 25 0
@@
 encoding utf-8
 Sheet 2 7
-Title ""
-Date ""
-Rev ""
-Comp ""
+Title "DK60TP"
+Date "2017-10-14"
+Rev "B"
+Comp "DarKou.fr"
 Comment1 ""
 Comment2 ""
@@
 F 1 "10uF" H 1110 1520 50  0000 L CNN
 F 2 "Capacitors_SMD:C_0805_HandSoldering" H 1100 1600 50  0001 C CNN
-F 3 "" H 1100 1600 50  0000 C CNN
+F 3 "http://www.mouser.com/ds/2/447/Yageo_UPY-GP_NP0_16V-to-50V_9-358835.pdf" H 1100 1600 50  0001 C CNN
+F 4 "CC0805ZKY5V7BB106" H 1100 1600 60  0001 C CNN "manf#"
 	1    1100 1600
 	1    0    0    1
@@
 F 1 "PAM2804" H 2450 1100 60  0000 C CNN
 F 2 "Footprint:SOT-23-5" H 2450 1350 60  0001 C CNN
-F 3 "" H 2450 1350 60  0000 C CNN
+F 3 "http://www.mouser.com/ds/2/115/PAM2804-247271.pdf" H 2450 1350 60  0001 C CNN
+F 4 "PAM2804AAB010" H 2450 1300 60  0001 C CNN "manf#"
 	1    2450 1300
 	1    0    0    -1
@@
 U 1 1 5932EA3C
 P 3250 1200
+AR Path="/5932EA3C" Ref="L1"  Part="1"
+AR Path="/5932D4E4/5932EA3C" Ref="L1"  Part="1"
 F 0 "L1" V 3200 1200 40  0000 C CNN
 F 1 "4.7uH" V 3350 1200 40  0000 C CNN
 F 2 "Footprint:Inductor_Bourn_4mmx4mm" H 3250 1200 60  0001 C CNN
-F 3 "" H 3250 1200 60  0000 C CNN
+F 3 "http://www.mouser.com/ds/2/445/744766904-709959.pdf" H 3250 1200 60  0001 C CNN
+F 4 "744766904" V 3250 1200 60  0001 C CNN "manf#"
 	1    3250 1200
 	0    -1   -1   0
@@
 F 1 "10uF" H 3910 1320 50  0000 L CNN
 F 2 "Capacitors_SMD:C_0805_HandSoldering" H 3900 1400 50  0001 C CNN
-F 3 "" H 3900 1400 50  0000 C CNN
+F 3 "http://www.mouser.com/ds/2/447/Yageo_UPY-GP_NP0_16V-to-50V_9-358835.pdf" H 3900 1400 50  0001 C CNN
+F 4 "CC0805ZKY5V7BB106" H 3900 1400 60  0001 C CNN "manf#"
 	1    3900 1400
 	1    0    0    1
@@
 F 1 "0.5" V 3450 1400 50  0000 C CNN
 F 2 "Resistors_SMD:R_0805_HandSoldering" V 3380 1400 50  0001 C CNN
-F 3 "" H 3450 1400 50  0000 C CNN
+F 3 "http://www.mouser.com/ds/2/447/PYu-RL_Group_521_RoHS_L_2-1131815.pdf" H 3450 1400 50  0001 C CNN
+F 4 "RL0805FR-7W0R5L" V 3450 1400 60  0001 C CNN "manf#"
 	1    3450 1400
 	0    1    1    0
