File: Kicad/BACKLIT.sch (KiCad schematic (older format))
At the start: 90 parts, among them U1 PAM2804

Commit message: - Some changes (routing/ground area/space)
- Updated routing
- Increased ground area
- Invert Split space 2.75U/2.25U
- Added missing led for backlit
Parts:
- added BL643: LED, Footprint:LED_TH_BIVAR, symbol LED
Connections:
- net LED_AN: now also BL643.2 (A)
- net LED_CATH: now also BL643.1 (K)
Changed lines of the file:
@@
 EESchema Schematic File Version 2
 LIBS:keyboard_parts
+LIBS:DK60TP-cache
 EELAYER 25 0
 EELAYER END
@@
 Connection ~ 1850 4600
 Wire Wire Line
-	1650 4900 6950 4900
+	1650 4900 7250 4900
 Connection ~ 1850 4900
 Connection ~ 2150 4900
@@
 Connection ~ 6050 4900
 Wire Wire Line
-	1650 5250 6950 5250
+	1650 5250 7250 5250
 Wire Wire Line
 	6350 5250 6350 5200
@@
 Connection ~ 4850 5900
 Connection ~ 4850 5550
+$Comp
+L LED BL643
+U 1 1 59E61F62
+P 7250 5050
+F 0 "BL643" H 7250 5150 50  0000 C CNN
+F 1 "LED" H 7250 4950 50  0001 C CNN
+F 2 "Footprint:LED_TH_BIVAR" H 7250 5050 50  0001 C CNN
+F 3 "" H 7250 5050 50  0000 C CNN
+	1    7250 5050
+	0    -1   -1   0
+$EndComp
+Connection ~ 6950 4900
+Wire Wire Line
+	7250 5250 7250 5200
+Connection ~ 6950 5250
 $EndSCHEMATC
