File: Kicad/BACKLIT.sch (KiCad schematic (older format))
At the start: 91 parts, among them U1 PAM2804

Commit message: - Added missing led for ivan ivanovitch layout
Parts:
- added BL423: LED, Footprint:LED_TH_BIVAR, symbol LED
Connections:
- net LED_AN: now also BL423.2 (A)
- net LED_CATH: now also BL423.1 (K)
Changed lines of the file:
@@
 	900  650  4200 650
 Wire Wire Line
-	1650 4250 6650 4250
+	1650 4250 6950 4250
 Wire Wire Line
-	1650 4600 6650 4600
+	1650 4600 6950 4600
 Connection ~ 6650 4900
 Wire Wire Line
@@
 	7250 5250 7250 5200
 Connection ~ 6950 5250
+$Comp
+L LED BL423
+U 1 1 59ECE45F
+P 6950 4400
+F 0 "BL423" H 6950 4500 50  0000 C CNN
+F 1 "LED" H 6950 4300 50  0001 C CNN
+F 2 "Footprint:LED_TH_BIVAR" H 6950 4400 50  0001 C CNN
+F 3 "" H 6950 4400 50  0000 C CNN
+	1    6950 4400
+	0    -1   -1   0
+$EndComp
+Connection ~ 6650 4250
+Wire Wire Line
+	6950 4600 6950 4550
+Connection ~ 6650 4600
 $EndSCHEMATC
