File: Kicad/Function_leds.sch (KiCad schematic (older format))
At the start: 2 parts

Commit message: - Updated 3 pin header for caps lock
Parts:
- added J3: CAPS_LOCK, Pin_Headers:Pin_Header_Angled_1x03, symbol 3PIN
Connections:
- net GND: now also J3.3
- net at LD1.2 (A): now also J3.2; no longer R6.2
- new net: J3.1, R6.2
Changed lines of the file:
@@
 	1600 1400 1900 1400
-Wire Wire Line
-	2200 1400 2500 1400
 Wire Wire Line
 	2800 1400 3150 1400
@@
 	900  1100 3400 1100
 Wire Notes Line
-	3400 1100 3400 2000
+	3400 1100 3400 2300
 Wire Notes Line
-	3400 2000 900  2000
+	900  1100 900  2300
+$Comp
+L 3PIN J3
+U 1 1 594A7AA3
+P 2400 2050
+F 0 "J3" H 2350 2250 60  0000 C CNN
+F 1 "CAPS_LOCK" H 2350 1850 60  0000 C CNN
+F 2 "Pin_Headers:Pin_Header_Angled_1x03" H 2400 2050 60  0001 C CNN
+F 3 "" H 2400 2050 60  0000 C CNN
+	1    2400 2050
+	0    -1   -1   0
+$EndComp
+Wire Wire Line
+	3150 1600 2500 1600
+Wire Wire Line
+	2500 1600 2500 1850
+Connection ~ 3150 1600
+Wire Wire Line
+	2500 1400 2400 1400
+Wire Wire Line
+	2400 1400 2400 1850
+Wire Wire Line
+	2200 1400 2300 1400
+Wire Wire Line
+	2300 1400 2300 1850
 Wire Notes Line
-	900  2000 900  1100
+	900  2300 3400 2300
 $EndSCHEMATC

Commit message: - First draw for Rev. B
Parts:
- J3: footprint Pin_Headers:Pin_Header_Angled_1x03 -> Pin_Headers:Pin_Header_Angled_1x03_Pitch2.54mm
Changed lines of the file:
@@
 F 0 "J3" H 2350 2250 60  0000 C CNN
 F 1 "CAPS_LOCK" H 2350 1850 60  0000 C CNN
-F 2 "Pin_Headers:Pin_Header_Angled_1x03" H 2400 2050 60  0001 C CNN
+F 2 "Pin_Headers:Pin_Header_Angled_1x03_Pitch2.54mm" H 2400 2050 60  0001 C CNN
 F 3 "" H 2400 2050 60  0000 C CNN
 	1    2400 2050

Commit message: Removed useless libraries
Merging all components in one library file to simplify maintenance
Parts:
- J3: manf# (none) -> 61300311021
- LD1: manf# (none) -> LR T68F-U1AA-1-1-Z
- R6: manf# (none) -> CR0805-FX-4701ELF
Changed lines of the file:
@@
 EESchema Schematic File Version 2
-LIBS:74xgxx
-LIBS:74xx
-LIBS:ac-dc
-LIBS:actel
-LIBS:adc-dac
-LIBS:allegro
-LIBS:Altera
-LIBS:analog_devices
-LIBS:analog_switches
-LIBS:audio
-LIBS:battery_management
-LIBS:bbd
-LIBS:bosch
-LIBS:brooktre
-LIBS:cmos4000
-LIBS:cmos_ieee
-LIBS:conn
-LIBS:contrib
-LIBS:cypress
-LIBS:dc-dc
-LIBS:device
-LIBS:digital-audio
-LIBS:diode
-LIBS:display
-LIBS:dsp
-LIBS:elec-unifil
-LIBS:ESD_Protection
-LIBS:ftdi
-LIBS:gennum
-LIBS:graphic_symbols
-LIBS:hc11
-LIBS:infineon
-LIBS:intel
-LIBS:interface
-LIBS:intersil
-LIBS:ir
-LIBS:Lattice
-LIBS:leds
-LIBS:LEM
-LIBS:linear
-LIBS:logic_programmable
-LIBS:maxim
-LIBS:mechanical
-LIBS:memory
-LIBS:microchip
-LIBS:microchip_dspic33dsc
-LIBS:microchip_pic10mcu
-LIBS:microchip_pic12mcu
-LIBS:microchip_pic16mcu
-LIBS:microchip_pic18mcu
-LIBS:microchip_pic24mcu
-LIBS:microchip_pic32mcu
-LIBS:microcontrollers
-LIBS:modules
-LIBS:motor_drivers
-LIBS:motorola
-LIBS:motors
-LIBS:msp430
-LIBS:nordicsemi
-LIBS:nxp
-LIBS:nxp_armmcu
-LIBS:onsemi
-LIBS:opto
-LIBS:Oscillators
-LIBS:philips
-LIBS:power
-LIBS:powerint
-LIBS:Power_Management
-LIBS:pspice
-LIBS:references
-LIBS:regul
-LIBS:relays
-LIBS:rfcom
-LIBS:RFSolutions
-LIBS:sensors
-LIBS:silabs
-LIBS:siliconi
-LIBS:stm8
-LIBS:stm32
-LIBS:supertex
-LIBS:switches
-LIBS:texas
-LIBS:transf
-LIBS:transistors
-LIBS:triac_thyristor
-LIBS:ttl_ieee
-LIBS:valves
-LIBS:video
-LIBS:wiznet
-LIBS:Xicor
-LIBS:xilinx
-LIBS:zetex
-LIBS:Zilog
 LIBS:keyboard_parts
-LIBS:mkl27z256vfm4
-LIBS:Trackpad
-LIBS:TS65
 LIBS:DK60TP-cache
 EELAYER 25 0
@@
 encoding utf-8
 Sheet 3 7
-Title ""
-Date ""
-Rev ""
-Comp ""
+Title "DK60TP"
+Date "2017-10-14"
+Rev "B"
+Comp "DarKou.fr"
 Comment1 ""
 Comment2 ""
@@
 F 1 "CAPS_LED" H 2650 1300 50  0000 C CNN
 F 2 "LEDs:LED_PLCC_2835" H 2650 1400 50  0001 C CNN
-F 3 "" H 2650 1400 50  0001 C CNN
+F 3 "http://www.mouser.com/ds/2/311/LR%20T68F%20-%20TOPLED-318599.pdf" H 2650 1400 50  0001 C CNN
+F 4 "LR T68F-U1AA-1-1-Z" H 2650 1400 60  0001 C CNN "manf#"
 	1    2650 1400
 	-1   0    0    1
@@
 F 1 "R" V 2050 1400 50  0000 C CNN
 F 2 "Resistors_SMD:R_0805_HandSoldering" V 1980 1400 50  0001 C CNN
-F 3 "" H 2050 1400 50  0001 C CNN
+F 3 "http://www.mouser.com/ds/2/54/chpreztr-977002.pdf" H 2050 1400 50  0001 C CNN
+F 4 "CR0805-FX-4701ELF" V 2050 1400 60  0001 C CNN "manf#"
 	1    2050 1400
 	0    -1   -1   0
@@
 F 1 "CAPS_LOCK" H 2350 1850 60  0000 C CNN
 F 2 "Pin_Headers:Pin_Header_Angled_1x03_Pitch2.54mm" H 2400 2050 60  0001 C CNN
-F 3 "" H 2400 2050 60  0000 C CNN
+F 3 "http://www.mouser.com/ds/2/445/6130xx11021-538004.pdf" H 2400 2050 60  0001 C CNN
+F 4 "61300311021" H 2400 2050 60  0001 C CNN "manf#"
 	1    2400 2050
 	0    -1   -1   0
