File: Kicad/HOLES.sch (KiCad schematic (older format))
At the start: 13 parts

Commit message: - First draw for Rev. B
Parts:
- added 6-6.25U_0: 6U/6.25U, Footprint:MXST, symbol MOUNT_HOLE
- added 6-7U_0: 6U/7U, Footprint:MXST, symbol MOUNT_HOLE
- added 6.25U_0: 6.25U, Footprint:MXST, symbol MOUNT_HOLE
- added 7U_0: 7U, Footprint:MXST, symbol MOUNT_HOLE
- added BACKSPACE_0, BACKSPACE_1: BACKSPACE, Footprint:MXST, symbol MOUNT_HOLE
- added ENTER_ANSI_0, ENTER_ANSI_1: ENTER_ANSI, Footprint:MXST, symbol MOUNT_HOLE
- added ENTER_ISO_0, ENTER_ISO_1: ENTER_ISO, Footprint:MXST, symbol MOUNT_HOLE
- added L_SHIFT_0, L_SHIFT_1: L_SHIFT, Footprint:MXST, symbol MOUNT_HOLE
- added R_SHIFT_0, R_SHIFT_1: R_SHIFT, Footprint:MXST, symbol MOUNT_HOLE
Other:
- moved on the sheet: MH4, MH7
Changed lines of the file:
@@
 L MOUNT_HOLE MH4
 U 1 1 593988C5
-P 3800 2250
-F 0 "MH4" H 3800 2400 60  0000 C CNN
-F 1 "BOTTOM_RIGHT" H 3800 2100 60  0000 C CNN
-F 2 "Footprint:Poker_oval_hole" H 3800 2250 60  0001 C CNN
-F 3 "" H 3800 2250 60  0000 C CNN
-	1    3800 2250
+P 3700 2700
+F 0 "MH4" H 3700 2850 60  0000 C CNN
+F 1 "BOTTOM_RIGHT" H 3700 2550 60  0000 C CNN
+F 2 "Footprint:Poker_oval_hole" H 3700 2700 60  0001 C CNN
+F 3 "" H 3700 2700 60  0000 C CNN
+	1    3700 2700
 	1    0    0    -1
 $EndComp
@@
 L MOUNT_HOLE MH7
 U 1 1 5939936E
-P 2700 2600
-F 0 "MH7" H 2700 2750 60  0000 C CNN
-F 1 "TRACKPOINT" H 2700 2450 60  0000 C CNN
-F 2 "Mounting_Holes:MountingHole_6mm" H 2700 2600 60  0001 C CNN
-F 3 "" H 2700 2600 60  0000 C CNN
-	1    2700 2600
+P 3250 2100
+F 0 "MH7" H 3250 2250 60  0000 C CNN
+F 1 "TRACKPOINT" H 3250 1950 60  0000 C CNN
+F 2 "Mounting_Holes:MountingHole_6mm" H 3250 2100 60  0001 C CNN
+F 3 "" H 3250 2100 60  0000 C CNN
+	1    3250 2100
 	1    0    0    -1
 $EndComp
@@
 	1    0    0    -1
 $EndComp
+$Comp
+L MOUNT_HOLE BACKSPACE_1
+U 1 1 59F193B9
+P 7050 2350
+F 0 "BACKSPACE_1" H 7050 2500 60  0000 C CNN
+F 1 "BACKSPACE" H 7050 2200 60  0000 C CNN
+F 2 "Footprint:MXST" H 7050 2350 60  0001 C CNN
+F 3 "" H 7050 2350 60  0000 C CNN
+	1    7050 2350
+	1    0    0    -1
+$EndComp
+$Comp
+L MOUNT_HOLE ENTER_ISO_0
+U 1 1 59F194E3
+P 6350 2850
+F 0 "ENTER_ISO_0" H 6350 3000 60  0000 C CNN
+F 1 "ENTER_ISO" H 6350 2700 60  0000 C CNN
+F 2 "Footprint:MXST" H 6350 2850 60  0001 C CNN
+F 3 "" H 6350 2850 60  0000 C CNN
+	1    6350 2850
+	1    0    0    -1
+$EndComp
+$Comp
+L MOUNT_HOLE ENTER_ANSI_0
+U 1 1 59F19575
+P 6350 3350
+F 0 "ENTER_ANSI_0" H 6350 3500 60  0000 C CNN
+F 1 "ENTER_ANSI" H 6350 3200 60  0000 C CNN
+F 2 "Footprint:MXST" H 6350 3350 60  0001 C CNN
+F 3 "" H 6350 3350 60  0000 C CNN
+	1    6350 3350
+	1    0    0    -1
+$EndComp
+$Comp
+L MOUNT_HOLE L_SHIFT_0
+U 1 1 59F1964D
+P 6350 3850
+F 0 "L_SHIFT_0" H 6350 4000 60  0000 C CNN
+F 1 "L_SHIFT" H 6350 3700 60  0000 C CNN
+F 2 "Footprint:MXST" H 6350 3850 60  0001 C CNN
+F 3 "" H 6350 3850 60  0000 C CNN
+	1    6350 3850
+	1    0    0    -1
+$EndComp
+$Comp
+L MOUNT_HOLE R_SHIFT_0
+U 1 1 59F1973A
+P 6350 4350
+F 0 "R_SHIFT_0" H 6350 4500 60  0000 C CNN
+F 1 "R_SHIFT" H 6350 4200 60  0000 C CNN
+F 2 "Footprint:MXST" H 6350 4350 60  0001 C CNN
+F 3 "" H 6350 4350 60  0000 C CNN
+	1    6350 4350
+	1    0    0    -1
+$EndComp
+$Comp
+L MOUNT_HOLE BACKSPACE_0
+U 1 1 59F19C51
+P 6350 2350
+F 0 "BACKSPACE_0" H 6350 2500 60  0000 C CNN
+F 1 "BACKSPACE" H 6350 2200 60  0000 C CNN
+F 2 "Footprint:MXST" H 6350 2350 60  0001 C CNN
+F 3 "" H 6350 2350 60  0000 C CNN
+	1    6350 2350
+	1    0    0    -1
+$EndComp
+$Comp
+L MOUNT_HOLE ENTER_ISO_1
+U 1 1 59F1A234
+P 7050 2850
+F 0 "ENTER_ISO_1" H 7050 3000 60  0000 C CNN
+F 1 "ENTER_ISO" H 7050 2700 60  0000 C CNN
+F 2 "Footprint:MXST" H 7050 2850 60  0001 C CNN
+F 3 "" H 7050 2850 60  0000 C CNN
+	1    7050 2850
+	1    0    0    -1
+$EndComp
+$Comp
+L MOUNT_HOLE ENTER_ANSI_1
+U 1 1 59F1A326
+P 7050 3350
+F 0 "ENTER_ANSI_1" H 7050 3500 60  0000 C CNN
+F 1 "ENTER_ANSI" H 7050 3200 60  0000 C CNN
+F 2 "Footprint:MXST" H 7050 3350 60  0001 C CNN
+F 3 "" H 7050 3350 60  0000 C CNN
+	1    7050 3350
+	1    0    0    -1
+$EndComp
+$Comp
+L MOUNT_HOLE L_SHIFT_1
+U 1 1 59F1AE1F
+P 7050 3850
+F 0 "L_SHIFT_1" H 7050 4000 60  0000 C CNN
+F 1 "L_SHIFT" H 7050 3700 60  0000 C CNN
+F 2 "Footprint:MXST" H 7050 3850 60  0001 C CNN
+F 3 "" H 7050 3850 60  0000 C CNN
+	1    7050 3850
+	1    0    0    -1
+$EndComp
+$Comp
+L MOUNT_HOLE R_SHIFT_1
+U 1 1 59F1AF2D
+P 7050 4350
+F 0 "R_SHIFT_1" H 7050 4500 60  0000 C CNN
+F 1 "R_SHIFT" H 7050 4200 60  0000 C CNN
+F 2 "Footprint:MXST" H 7050 4350 60  0001 C CNN
+F 3 "" H 7050 4350 60  0000 C CNN
+	1    7050 4350
+	1    0    0    -1
+$EndComp
+$Comp
+L MOUNT_HOLE 6.25U_0
+U 1 1 59F1B788
+P 6350 4850
+F 0 "6.25U_0" H 6350 5000 60  0000 C CNN
+F 1 "6.25U" H 6350 4700 60  0000 C CNN
+F 2 "Footprint:MXST" H 6350 4850 60  0001 C CNN
+F 3 "" H 6350 4850 60  0000 C CNN
+	1    6350 4850
+	1    0    0    -1
+$EndComp
+$Comp
+L MOUNT_HOLE 6-7U_0
+U 1 1 59F1B850
+P 7050 4850
+F 0 "6-7U_0" H 7050 5000 60  0000 C CNN
+F 1 "6U/7U" H 7050 4700 60  0000 C CNN
+F 2 "Footprint:MXST" H 7050 4850 60  0001 C CNN
+F 3 "" H 7050 4850 60  0000 C CNN
+	1    7050 4850
+	1    0    0    -1
+$EndComp
+$Comp
+L MOUNT_HOLE 6-6.25U_0
+U 1 1 59F1B954
+P 6350 5350
+F 0 "6-6.25U_0" H 6350 5500 60  0000 C CNN
+F 1 "6U/6.25U" H 6350 5200 60  0000 C CNN
+F 2 "Footprint:MXST" H 6350 5350 60  0001 C CNN
+F 3 "" H 6350 5350 60  0000 C CNN
+	1    6350 5350
+	1    0    0    -1
+$EndComp
+$Comp
+L MOUNT_HOLE 7U_0
+U 1 1 59F1B9E0
+P 7050 5350
+F 0 "7U_0" H 7050 5500 60  0000 C CNN
+F 1 "7U" H 7050 5200 60  0000 C CNN
+F 2 "Footprint:MXST" H 7050 5350 60  0001 C CNN
+F 3 "" H 7050 5350 60  0000 C CNN
+	1    7050 5350
+	1    0    0    -1
+$EndComp

Commit message: - First commit for splitted spacebar
Parts:
- added SPC_225_0: SPC_225_0, Footprint:MXST, symbol MOUNT_HOLE
- added SPC_275_0: SPC_275_0, Footprint:MXST, symbol MOUNT_HOLE
- added SPC_275_1: SPC_275_1, Footprint:MXST, symbol MOUNT_HOLE
Changed lines of the file:
@@
+	1    0    0    -1
+$EndComp
+$Comp
+L MOUNT_HOLE SPC_275_0
+U 1 1 59DE9C95
+P 6350 5850
+F 0 "SPC_275_0" H 6350 6000 60  0000 C CNN
+F 1 "SPC_275_0" H 6350 5700 60  0000 C CNN
+F 2 "Footprint:MXST" H 6350 5850 60  0001 C CNN
+F 3 "" H 6350 5850 60  0000 C CNN
+	1    6350 5850
+	1    0    0    -1
+$EndComp
+$Comp
+L MOUNT_HOLE SPC_275_1
+U 1 1 59DE9D0D
+P 7050 5850
+F 0 "SPC_275_1" H 7050 6000 60  0000 C CNN
+F 1 "SPC_275_1" H 7050 5700 60  0000 C CNN
+F 2 "Footprint:MXST" H 7050 5850 60  0001 C CNN
+F 3 "" H 7050 5850 60  0000 C CNN
+	1    7050 5850
+	1    0    0    -1
+$EndComp
+$Comp
+L MOUNT_HOLE SPC_225_0
+U 1 1 59DE9D8E
+P 6350 6350
+F 0 "SPC_225_0" H 6350 6500 60  0000 C CNN
+F 1 "SPC_225_0" H 6350 6200 60  0000 C CNN
+F 2 "Footprint:MXST" H 6350 6350 60  0001 C CNN
+F 3 "" H 6350 6350 60  0000 C CNN
+	1    6350 6350
 	1    0    0    -1
 $EndComp
