File: Kicad/HOLES.sch (KiCad schematic (older format))
At the start: 30 parts

Commit message: - Some changes (routing/ground area/space)
- Updated routing
- Increased ground area
- Invert Split space 2.75U/2.25U
- Added missing led for backlit
Parts:
- removed SPC_275_1: SPC_275_1, Footprint:MXST, symbol MOUNT_HOLE
- added SPC_R_SPLIT_1: SPC_275_1, Footprint:MXST, symbol MOUNT_HOLE
- SPC_R_SPLIT_0: renamed from SPC_225_0; value SPC_225_0 -> SPC_275_0
Changed lines of the file:
@@
 EESchema Schematic File Version 2
 LIBS:keyboard_parts
+LIBS:DK60TP-cache
 EELAYER 25 0
 EELAYER END
@@
 $EndComp
 $Comp
-L MOUNT_HOLE SPC_275_1
-U 1 1 59DE9D0D
-P 7050 5850
-F 0 "SPC_275_1" H 7050 6000 60  0000 C CNN
-F 1 "SPC_275_1" H 7050 5700 60  0000 C CNN
-F 2 "Footprint:MXST" H 7050 5850 60  0001 C CNN
-F 3 "" H 7050 5850 60  0000 C CNN
-	1    7050 5850
-	1    0    0    -1
-$EndComp
-$Comp
-L MOUNT_HOLE SPC_225_0
+L MOUNT_HOLE SPC_R_SPLIT_0
 U 1 1 59DE9D8E
 P 6350 6350
-F 0 "SPC_225_0" H 6350 6500 60  0000 C CNN
-F 1 "SPC_225_0" H 6350 6200 60  0000 C CNN
+F 0 "SPC_R_SPLIT_0" H 6350 6500 60  0000 C CNN
+F 1 "SPC_275_0" H 6350 6200 60  0000 C CNN
 F 2 "Footprint:MXST" H 6350 6350 60  0001 C CNN
 F 3 "" H 6350 6350 60  0000 C CNN
@@
 	1    0    0    -1
 $EndComp
+$Comp
+L MOUNT_HOLE SPC_R_SPLIT_1
+U 1 1 59E6511D
+P 7050 6350
+F 0 "SPC_R_SPLIT_1" H 7050 6500 60  0000 C CNN
+F 1 "SPC_275_1" H 7050 6200 60  0000 C CNN
+F 2 "Footprint:MXST" H 7050 6350 60  0001 C CNN
+F 3 "" H 7050 6350 60  0000 C CNN
+	1    7050 6350
+	1    0    0    -1
+$EndComp
