File: Kicad/HOLES.sch (KiCad schematic (older format))
At the start: 30 parts

Commit message: - Fixed some bugs
* Fixed bug when trying to show 3D Viewer (bad egde cuts)
* Updated GND areas
* Fixed error when loading net list (bad chip name for holes)
Parts:
- 6-6.25U_0, 6-7U_0, 6.25U_0, 7U_0, BACKSPACE_0, BACKSPACE_1, ENTER_ANSI_0, ENTER_ANSI_1, ENTER_ISO_0, ENTER_ISO_1, L_SHIFT_0, L_SHIFT_1, MH1, MH10, MH11, MH12, MH13, MH2, MH3, MH4, MH5, MH6, MH7, MH8, MH9, R_SHIFT_0, R_SHIFT_1, SPC_275_0, SPC_R_SPLIT_0, SPC_R_SPLIT_1: symbol MOUNT_HOLE -> MISC

Commit message: - Added ivan ivanovitch layout
Parts:
- added 7U_LEFT_0: 7U_LEFT_0, Footprint:MXST, symbol MISC
Changed lines of the file:
@@
 EESchema Schematic File Version 2
 LIBS:kicad_parts
-LIBS:DK60TP-cache
 EELAYER 25 0
 EELAYER END
@@
 	1    0    0    -1
 $EndComp
+$Comp
+L MISC 7U_LEFT_0
+U 1 1 59EC8135
+P 6800 4100
+F 0 "7U_LEFT_0" H 6800 4250 60  0000 C CNN
+F 1 "7U_LEFT_0" H 6800 3950 60  0000 C CNN
+F 2 "Footprint:MXST" H 6800 4100 60  0001 C CNN
+F 3 "" H 6800 4100 60  0000 C CNN
+	1    6800 4100
+	1    0    0    -1
+$EndComp
