File: Kicad/RGB_UNDERGLOW.sch (KiCad schematic (older format))
At the start: 11 parts, among them J2 RGB

Commit message: - First draw for Rev. B
Parts:
- added CRGB5, CRGB6, CRGB7: 0.1u, Capacitors_SMD:C_0805_HandSoldering, symbol C_Small
- added RGB5, RGB6, RGB7: WS2812B, Footprint:WS2812B, symbol WS2812B
- renumbered C12 to CRGB0, C13 to CRGB1, C14 to CRGB2, C15 to CRGB3, C16 to CRGB4, D149 to RGB0, D150 to RGB1, D151 to RGB2, D152 to RGB3, D153 to RGB4
Connections:
- net DOUT: now also RGB7.2 (DOUT); no longer RGB4.2 (DOUT)
- net GND: now also CRGB5.2, CRGB6.2, CRGB7.2, RGB5.3 (VSS), RGB6.3 (VSS), RGB7.3 (VSS)
- net VCC: now also CRGB5.1, CRGB6.1, CRGB7.1, RGB5.1 (VDD), RGB6.1 (VDD), RGB7.1 (VDD)
- new net: RGB4.2 (DOUT), RGB5.4 (DIN)
- new net: RGB5.2 (DOUT), RGB6.4 (DIN)
- new net: RGB6.2 (DOUT), RGB7.4 (DIN)
Changed lines of the file:
@@
 $EndComp
 $Comp
-L WS2812B D149
+L WS2812B RGB0
 U 1 1 593558EF
 P 2700 1450
-F 0 "D149" H 2550 1650 50  0000 L CNN
-F 1 "WS2812B" H 2500 1250 50  0000 L CNN
+F 0 "RGB0" H 2550 1650 50  0000 L CNN
+F 1 "WS2812B" H 2500 1250 50  0001 L CNN
 F 2 "Footprint:WS2812B" H 2700 1450 50  0001 L CNN
 F 3 "" H 2700 1450 60  0000 C CNN
@@
 RGB
 $Comp
-L C_Small C12
+L C_Small CRGB0
 U 1 1 5935598D
 P 1950 1600
-F 0 "C12" H 1960 1670 50  0000 L CNN
+F 0 "CRGB0" H 1960 1670 50  0001 L CNN
 F 1 "0.1u" H 1960 1520 50  0000 L CNN
 F 2 "Capacitors_SMD:C_0805_HandSoldering" H 1950 1600 50  0001 C CNN
@@
 $EndComp
 $Comp
-L WS2812B D150
+L WS2812B RGB1
 U 1 1 59355B4F
 P 2700 2050
-F 0 "D150" H 2550 2250 50  0000 L CNN
-F 1 "WS2812B" H 2500 1850 50  0000 L CNN
+F 0 "RGB1" H 2550 2250 50  0000 L CNN
+F 1 "WS2812B" H 2500 1850 50  0001 L CNN
 F 2 "Footprint:WS2812B" H 2700 2050 50  0001 L CNN
 F 3 "" H 2700 2050 60  0000 C CNN
@@
 $EndComp
 $Comp
-L WS2812B D151
+L WS2812B RGB2
 U 1 1 59355BD6
 P 2700 2650
-F 0 "D151" H 2550 2850 50  0000 L CNN
-F 1 "WS2812B" H 2500 2450 50  0000 L CNN
+F 0 "RGB2" H 2550 2850 50  0000 L CNN
+F 1 "WS2812B" H 2500 2450 50  0001 L CNN
 F 2 "Footprint:WS2812B" H 2700 2650 50  0001 L CNN
 F 3 "" H 2700 2650 60  0000 C CNN
@@
 $EndComp
 $Comp
-L WS2812B D152
+L WS2812B RGB3
 U 1 1 59355D9F
 P 2700 3250
-F 0 "D152" H 2550 3450 50  0000 L CNN
-F 1 "WS2812B" H 2500 3050 50  0000 L CNN
+F 0 "RGB3" H 2550 3450 50  0000 L CNN
+F 1 "WS2812B" H 2500 3050 50  0001 L CNN
 F 2 "Footprint:WS2812B" H 2700 3250 50  0001 L CNN
 F 3 "" H 2700 3250 60  0000 C CNN
@@
 $EndComp
 $Comp
-L WS2812B D153
+L WS2812B RGB4
 U 1 1 59355E07
 P 2700 3850
-F 0 "D153" H 2550 4050 50  0000 L CNN
-F 1 "WS2812B" H 2500 3650 50  0000 L CNN
+F 0 "RGB4" H 2550 4050 50  0000 L CNN
+F 1 "WS2812B" H 2500 3650 50  0001 L CNN
 F 2 "Footprint:WS2812B" H 2700 3850 50  0001 L CNN
 F 3 "" H 2700 3850 60  0000 C CNN
@@
 L GND #PWR021
 U 1 1 59355E8A
-P 3200 4100
-F 0 "#PWR021" H 3200 3850 50  0001 C CNN
-F 1 "GND" H 3200 3950 50  0000 C CNN
-F 2 "" H 3200 4100 50  0000 C CNN
-F 3 "" H 3200 4100 50  0000 C CNN
-	1    3200 4100
-	1    0    0    -1
-$EndComp
-$Comp
-L C_Small C13
+P 3200 6000
+F 0 "#PWR021" H 3200 5750 50  0001 C CNN
+F 1 "GND" H 3200 5850 50  0000 C CNN
+F 2 "" H 3200 6000 50  0000 C CNN
+F 3 "" H 3200 6000 50  0000 C CNN
+	1    3200 6000
+	1    0    0    -1
+$EndComp
+$Comp
+L C_Small CRGB1
 U 1 1 59356319
 P 1950 2200
-F 0 "C13" H 1960 2270 50  0000 L CNN
+F 0 "CRGB1" H 1960 2270 50  0001 L CNN
 F 1 "0.1u" H 1960 2120 50  0000 L CNN
 F 2 "Capacitors_SMD:C_0805_HandSoldering" H 1950 2200 50  0001 C CNN
@@
 $EndComp
 $Comp
-L C_Small C14
+L C_Small CRGB2
 U 1 1 5935635E
 P 1950 2800
-F 0 "C14" H 1960 2870 50  0000 L CNN
+F 0 "CRGB2" H 1960 2870 50  0001 L CNN
 F 1 "0.1u" H 1960 2720 50  0000 L CNN
 F 2 "Capacitors_SMD:C_0805_HandSoldering" H 1950 2800 50  0001 C CNN
@@
 $EndComp
 $Comp
-L C_Small C15
+L C_Small CRGB3
 U 1 1 593563A8
 P 1950 3400
-F 0 "C15" H 1960 3470 50  0000 L CNN
+F 0 "CRGB3" H 1960 3470 50  0001 L CNN
 F 1 "0.1u" H 1960 3320 50  0000 L CNN
 F 2 "Capacitors_SMD:C_0805_HandSoldering" H 1950 3400 50  0001 C CNN
@@
 $EndComp
 Wire Wire Line
-	1700 1100 1700 3750
+	1700 1100 1700 5550
 Wire Wire Line
 	1700 1350 2450 1350
@@
 	3050 3750 2950 3750
 Wire Wire Line
-	2950 3950 3200 3950
-Wire Wire Line
-	3200 1550 3200 4100
-Wire Wire Line
-	2950 2750 3200 2750
+	3200 3950 2950 3950
+Wire Wire Line
+	3200 2750 2950 2750
 Connection ~ 3200 3950
 Wire Wire Line
@@
 Connection ~ 3200 2750
 Wire Wire Line
-	2950 3350 3200 3350
+	3200 3350 2950 3350
 Connection ~ 3200 3350
 Wire Wire Line
@@
 Wire Wire Line
 	5450 2100 5450 2600
-Text GLabel 2550 4200 2    60   Input ~ 0
+Text GLabel 2550 5950 2    60   Input ~ 0
 DOUT
 Text GLabel 5200 2600 3    60   Input ~ 0
@@
 	5200 2200 5200 2600
 $Comp
-L C_Small C16
+L C_Small CRGB4
 U 1 1 5935745A
 P 1950 4000
-F 0 "C16" H 1960 4070 50  0000 L CNN
+F 0 "CRGB4" H 1960 4070 50  0001 L CNN
 F 1 "0.1u" H 1960 3920 50  0000 L CNN
 F 2 "Capacitors_SMD:C_0805_HandSoldering" H 1950 4000 50  0001 C CNN
@@
 Wire Wire Line
 	2450 3950 2350 3950
-Wire Wire Line
-	2350 3950 2350 4200
-Wire Wire Line
-	2350 4200 2550 4200
 Wire Wire Line
 	1950 3900 1950 3750
@@
 Text GLabel 4450 3250 2    60   Input ~ 0
 DOUT
+$Comp
+L WS2812B RGB5
+U 1 1 59EC4E8D
+P 2700 4450
+F 0 "RGB5" H 2550 4650 50  0000 L CNN
+F 1 "WS2812B" H 2500 4250 50  0001 L CNN
+F 2 "Footprint:WS2812B" H 2700 4450 50  0001 L CNN
+F 3 "" H 2700 4450 60  0000 C CNN
+	1    2700 4450
+	1    0    0    -1
+$EndComp
+Wire Wire Line
+	2350 3950 2350 4150
+Wire Wire Line
+	2350 4150 3050 4150
+Wire Wire Line
+	3050 4150 3050 4350
+Wire Wire Line
+	3050 4350 2950 4350
+Wire Wire Line
+	3200 4550 2950 4550
+Wire Wire Line
+	3200 1550 3200 6000
+Wire Wire Line
+	1700 4350 2450 4350
+Wire Wire Line
+	2350 4750 3050 4750
+Wire Wire Line
+	3050 4750 3050 4950
+Wire Wire Line
+	3050 4950 2950 4950
+$Comp
+L WS2812B RGB6
+U 1 1 59EC64F1
+P 2700 5050
+F 0 "RGB6" H 2550 5250 50  0000 L CNN
+F 1 "WS2812B" H 2500 4850 50  0001 L CNN
+F 2 "Footprint:WS2812B" H 2700 5050 50  0001 L CNN
+F 3 "" H 2700 5050 60  0000 C CNN
+	1    2700 5050
+	1    0    0    -1
+$EndComp
+Connection ~ 3200 5150
+Connection ~ 3200 4550
+Wire Wire Line
+	3200 5150 2950 5150
+Wire Wire Line
+	2450 5150 2350 5150
+Wire Wire Line
+	2350 5150 2350 5350
+Wire Wire Line
+	2350 5350 3050 5350
+Wire Wire Line
+	3050 5350 3050 5550
+Wire Wire Line
+	3050 5550 2950 5550
+$Comp
+L WS2812B RGB7
+U 1 1 59EC6A64
+P 2700 5650
+F 0 "RGB7" H 2550 5850 50  0000 L CNN
+F 1 "WS2812B" H 2500 5450 50  0001 L CNN
+F 2 "Footprint:WS2812B" H 2700 5650 50  0001 L CNN
+F 3 "" H 2700 5650 60  0000 C CNN
+	1    2700 5650
+	1    0    0    -1
+$EndComp
+Wire Wire Line
+	3200 5750 2950 5750
+Connection ~ 3200 5750
+Wire Wire Line
+	2450 5750 2350 5750
+Wire Wire Line
+	2350 5750 2350 5950
+Wire Wire Line
+	2350 5950 2550 5950
+Connection ~ 1700 3750
+Wire Wire Line
+	1700 4950 2450 4950
+Connection ~ 1700 4350
+Wire Wire Line
+	1700 5550 2450 5550
+Connection ~ 1700 4950
+$Comp
+L C_Small CRGB5
+U 1 1 59EC8437
+P 1950 4600
+F 0 "CRGB5" H 1960 4670 50  0001 L CNN
+F 1 "0.1u" H 1960 4520 50  0000 L CNN
+F 2 "Capacitors_SMD:C_0805_HandSoldering" H 1950 4600 50  0001 C CNN
+F 3 "" H 1950 4600 50  0000 C CNN
+	1    1950 4600
+	1    0    0    -1
+$EndComp
+Wire Wire Line
+	1950 4350 1950 4500
+Connection ~ 1950 4350
+$Comp
+L C_Small CRGB6
+U 1 1 59EC893A
+P 1950 5200
+F 0 "CRGB6" H 1960 5270 50  0001 L CNN
+F 1 "0.1u" H 1960 5120 50  0000 L CNN
+F 2 "Capacitors_SMD:C_0805_HandSoldering" H 1950 5200 50  0001 C CNN
+F 3 "" H 1950 5200 50  0000 C CNN
+	1    1950 5200
+	1    0    0    -1
+$EndComp
+Wire Wire Line
+	1950 4950 1950 5100
+Connection ~ 1950 4950
+$Comp
+L C_Small CRGB7
+U 1 1 59EC8E72
+P 1950 5800
+F 0 "CRGB7" H 1960 5870 50  0001 L CNN
+F 1 "0.1u" H 1960 5720 50  0000 L CNN
+F 2 "Capacitors_SMD:C_0805_HandSoldering" H 1950 5800 50  0001 C CNN
+F 3 "" H 1950 5800 50  0000 C CNN
+	1    1950 5800
+	1    0    0    -1
+$EndComp
+Wire Wire Line
+	1950 5550 1950 5700
+Connection ~ 1950 5550
+$Comp
+L GND #PWR029
+U 1 1 59EC95F1
+P 1950 4700
+F 0 "#PWR029" H 1950 4450 50  0001 C CNN
+F 1 "GND" H 1950 4550 50  0000 C CNN
+F 2 "" H 1950 4700 50  0000 C CNN
+F 3 "" H 1950 4700 50  0000 C CNN
+	1    1950 4700
+	1    0    0    -1
+$EndComp
+$Comp
+L GND #PWR030
+U 1 1 59EC962F
+P 1950 5300
+F 0 "#PWR030" H 1950 5050 50  0001 C CNN
+F 1 "GND" H 1950 5150 50  0000 C CNN
+F 2 "" H 1950 5300 50  0000 C CNN
+F 3 "" H 1950 5300 50  0000 C CNN
+	1    1950 5300
+	1    0    0    -1
+$EndComp
+$Comp
+L GND #PWR031
+U 1 1 59EC9D11
+P 1950 5900
+F 0 "#PWR031" H 1950 5650 50  0001 C CNN
+F 1 "GND" H 1950 5750 50  0000 C CNN
+F 2 "" H 1950 5900 50  0000 C CNN
+F 3 "" H 1950 5900 50  0000 C CNN
+	1    1950 5900
+	1    0    0    -1
+$EndComp
+Wire Wire Line
+	2450 4550 2350 4550
+Wire Wire Line
+	2350 4550 2350 4750
 $EndSCHEMATC

Commit message: Removed useless libraries
Merging all components in one library file to simplify maintenance
Parts:
- CRGB0, CRGB1, CRGB2, CRGB3, CRGB4, CRGB5, CRGB6, CRGB7: manf# (none) -> CC0805ZRY5V9BB104
- J2: manf# (none) -> 53048-0310
- RGB0, RGB1, RGB2, RGB3, RGB4, RGB5, RGB6, RGB7: manf# (none) -> COM-13667
Changed lines of the file:
@@
 EESchema Schematic File Version 2
-LIBS:74xgxx
-LIBS:74xx
-LIBS:ac-dc
-LIBS:actel
-LIBS:adc-dac
-LIBS:allegro
-LIBS:Altera
-LIBS:analog_devices
-LIBS:analog_switches
-LIBS:audio
-LIBS:battery_management
-LIBS:bbd
-LIBS:bosch
-LIBS:brooktre
-LIBS:cmos4000
-LIBS:cmos_ieee
-LIBS:conn
-LIBS:contrib
-LIBS:cypress
-LIBS:dc-dc
-LIBS:device
-LIBS:digital-audio
-LIBS:diode
-LIBS:display
-LIBS:dsp
-LIBS:elec-unifil
-LIBS:ESD_Protection
-LIBS:ftdi
-LIBS:gennum
-LIBS:graphic_symbols
-LIBS:hc11
-LIBS:infineon
-LIBS:intel
-LIBS:interface
-LIBS:intersil
-LIBS:ir
-LIBS:Lattice
-LIBS:leds
-LIBS:LEM
-LIBS:linear
-LIBS:logic_programmable
-LIBS:maxim
-LIBS:mechanical
-LIBS:memory
-LIBS:microchip
-LIBS:microchip_dspic33dsc
-LIBS:microchip_pic10mcu
-LIBS:microchip_pic12mcu
-LIBS:microchip_pic16mcu
-LIBS:microchip_pic18mcu
-LIBS:microchip_pic24mcu
-LIBS:microchip_pic32mcu
-LIBS:microcontrollers
-LIBS:modules
-LIBS:motor_drivers
-LIBS:motorola
-LIBS:motors
-LIBS:msp430
-LIBS:nordicsemi
-LIBS:nxp
-LIBS:nxp_armmcu
-LIBS:onsemi
-LIBS:opto
-LIBS:Oscillators
-LIBS:philips
-LIBS:power
-LIBS:powerint
-LIBS:Power_Management
-LIBS:pspice
-LIBS:references
-LIBS:regul
-LIBS:relays
-LIBS:rfcom
-LIBS:RFSolutions
-LIBS:sensors
-LIBS:silabs
-LIBS:siliconi
-LIBS:stm8
-LIBS:stm32
-LIBS:supertex
-LIBS:switches
-LIBS:texas
-LIBS:transf
-LIBS:transistors
-LIBS:triac_thyristor
-LIBS:ttl_ieee
-LIBS:valves
-LIBS:video
-LIBS:wiznet
-LIBS:Xicor
-LIBS:xilinx
-LIBS:zetex
-LIBS:Zilog
 LIBS:keyboard_parts
-LIBS:mkl27z256vfm4
-LIBS:Trackpad
-LIBS:TS65
 LIBS:DK60TP-cache
 EELAYER 25 0
@@
 encoding utf-8
 Sheet 6 7
-Title ""
-Date ""
-Rev ""
-Comp ""
+Title "DK60TP"
+Date "2017-10-14"
+Rev "B"
+Comp "DarKou.fr"
 Comment1 ""
 Comment2 ""
@@
 F 2 "Footprint:WS2812B" H 2700 1450 50  0001 L CNN
 F 3 "" H 2700 1450 60  0000 C CNN
+F 4 "COM-13667" H 2700 1450 60  0001 C CNN "manf#"
 	1    2700 1450
 	1    0    0    -1
@@
 F 1 "0.1u" H 1960 1520 50  0000 L CNN
 F 2 "Capacitors_SMD:C_0805_HandSoldering" H 1950 1600 50  0001 C CNN
-F 3 "" H 1950 1600 50  0000 C CNN
+F 3 "http://www.yageo.com/documents/recent/UPY-GPHC_Y5V_6.3V-to-50V_8.pdf" H 1950 1600 50  0001 C CNN
+F 4 "CC0805ZRY5V9BB104" H 1950 1600 60  0001 C CNN "manf#"
 	1    1950 1600
 	1    0    0    -1
@@
 F 2 "Footprint:WS2812B" H 2700 2050 50  0001 L CNN
 F 3 "" H 2700 2050 60  0000 C CNN
+F 4 "COM-13667" H 2700 2050 60  0001 C CNN "manf#"
 	1    2700 2050
 	1    0    0    -1
@@
 F 2 "Footprint:WS2812B" H 2700 2650 50  0001 L CNN
 F 3 "" H 2700 2650 60  0000 C CNN
+F 4 "COM-13667" H 2700 2650 60  0001 C CNN "manf#"
 	1    2700 2650
 	1    0    0    -1
@@
 F 2 "Footprint:WS2812B" H 2700 3250 50  0001 L CNN
 F 3 "" H 2700 3250 60  0000 C CNN
+F 4 "COM-13667" H 2700 3250 60  0001 C CNN "manf#"
 	1    2700 3250
 	1    0    0    -1
@@
 F 2 "Footprint:WS2812B" H 2700 3850 50  0001 L CNN
 F 3 "" H 2700 3850 60  0000 C CNN
+F 4 "COM-13667" H 2700 3850 60  0001 C CNN "manf#"
 	1    2700 3850
 	1    0    0    -1
@@
 F 1 "0.1u" H 1960 2120 50  0000 L CNN
 F 2 "Capacitors_SMD:C_0805_HandSoldering" H 1950 2200 50  0001 C CNN
-F 3 "" H 1950 2200 50  0000 C CNN
+F 3 "http://www.yageo.com/documents/recent/UPY-GPHC_Y5V_6.3V-to-50V_8.pdf" H 1950 2200 50  0001 C CNN
+F 4 "CC0805ZRY5V9BB104" H 1950 2200 60  0001 C CNN "manf#"
 	1    1950 2200
 	1    0    0    -1
@@
 F 1 "0.1u" H 1960 2720 50  0000 L CNN
 F 2 "Capacitors_SMD:C_0805_HandSoldering" H 1950 2800 50  0001 C CNN
-F 3 "" H 1950 2800 50  0000 C CNN
+F 3 "http://www.yageo.com/documents/recent/UPY-GPHC_Y5V_6.3V-to-50V_8.pdf" H 1950 2800 50  0001 C CNN
+F 4 "CC0805ZRY5V9BB104" H 1950 2800 60  0001 C CNN "manf#"
 	1    1950 2800
 	1    0    0    -1
@@
 F 1 "0.1u" H 1960 3320 50  0000 L CNN
 F 2 "Capacitors_SMD:C_0805_HandSoldering" H 1950 3400 50  0001 C CNN
-F 3 "" H 1950 3400 50  0000 C CNN
+F 3 "http://www.yageo.com/documents/recent/UPY-GPHC_Y5V_6.3V-to-50V_8.pdf" H 1950 3400 50  0001 C CNN
+F 4 "CC0805ZRY5V9BB104" H 1950 3400 60  0001 C CNN "manf#"
 	1    1950 3400
 	1    0    0    -1
@@
 F 1 "RGB" H 4400 1900 60  0000 C CNN
 F 2 "Connectors_Molex:Molex_PicoBlade_53048-0310_03x1.25mm_Angled" H 4450 2100 60  0001 C CNN
-F 3 "" H 4450 2100 60  0000 C CNN
+F 3 "http://www.mouser.com/ds/2/276/0530480310_PCB_HEADERS-171011.pdf" H 4450 2100 60  0001 C CNN
+F 4 "53048-0310" H 4450 2100 60  0001 C CNN "manf#"
 	1    4450 2100
 	1    0    0    -1
@@
 F 1 "0.1u" H 1960 3920 50  0000 L CNN
 F 2 "Capacitors_SMD:C_0805_HandSoldering" H 1950 4000 50  0001 C CNN
-F 3 "" H 1950 4000 50  0000 C CNN
+F 3 "http://www.yageo.com/documents/recent/UPY-GPHC_Y5V_6.3V-to-50V_8.pdf" H 1950 4000 50  0001 C CNN
+F 4 "CC0805ZRY5V9BB104" H 1950 4000 60  0001 C CNN "manf#"
 	1    1950 4000
 	1    0    0    -1
@@
 F 2 "Footprint:WS2812B" H 2700 4450 50  0001 L CNN
 F 3 "" H 2700 4450 60  0000 C CNN
+F 4 "COM-13667" H 2700 4450 60  0001 C CNN "manf#"
 	1    2700 4450
 	1    0    0    -1
@@
 F 2 "Footprint:WS2812B" H 2700 5050 50  0001 L CNN
 F 3 "" H 2700 5050 60  0000 C CNN
+F 4 "COM-13667" H 2700 5050 60  0001 C CNN "manf#"
 	1    2700 5050
 	1    0    0    -1
@@
 F 2 "Footprint:WS2812B" H 2700 5650 50  0001 L CNN
 F 3 "" H 2700 5650 60  0000 C CNN
+F 4 "COM-13667" H 2700 5650 60  0001 C CNN "manf#"
 	1    2700 5650
 	1    0    0    -1
@@
 F 1 "0.1u" H 1960 4520 50  0000 L CNN
 F 2 "Capacitors_SMD:C_0805_HandSoldering" H 1950 4600 50  0001 C CNN
-F 3 "" H 1950 4600 50  0000 C CNN
+F 3 "http://www.yageo.com/documents/recent/UPY-GPHC_Y5V_6.3V-to-50V_8.pdf" H 1950 4600 50  0001 C CNN
+F 4 "CC0805ZRY5V9BB104" H 1950 4600 60  0001 C CNN "manf#"
 	1    1950 4600
 	1    0    0    -1
@@
 F 1 "0.1u" H 1960 5120 50  0000 L CNN
 F 2 "Capacitors_SMD:C_0805_HandSoldering" H 1950 5200 50  0001 C CNN
-F 3 "" H 1950 5200 50  0000 C CNN
+F 3 "http://www.yageo.com/documents/recent/UPY-GPHC_Y5V_6.3V-to-50V_8.pdf" H 1950 5200 50  0001 C CNN
+F 4 "CC0805ZRY5V9BB104" H 1950 5200 60  0001 C CNN "manf#"
 	1    1950 5200
 	1    0    0    -1
@@
 F 1 "0.1u" H 1960 5720 50  0000 L CNN
 F 2 "Capacitors_SMD:C_0805_HandSoldering" H 1950 5800 50  0001 C CNN
-F 3 "" H 1950 5800 50  0000 C CNN
+F 3 "http://www.yageo.com/documents/recent/UPY-GPHC_Y5V_6.3V-to-50V_8.pdf" H 1950 5800 50  0001 C CNN
+F 4 "CC0805ZRY5V9BB104" H 1950 5800 60  0001 C CNN "manf#"
 	1    1950 5800
 	1    0    0    -1
