File: Kicad/TRACKPOINT.sch (KiCad schematic (older format))
At the start: 20 parts, among them P2 MAIN_BOARD, P3 TRACKPOINT

Commit message: - First draw for Rev. B
Parts:
- DK34: renamed from DM34; value D -> D43
- DK44: renamed from DM44; value D -> D44
- DK54: renamed from DM54; value D -> D45
- K341: renamed from KM341; value KEYSW -> LMB
- K541: renamed from KM541; value KEYSW -> RMB
- renumbered C19 to CRGB10, C17 to CRGB8, C18 to CRGB9, KM340 to K340, KM440 to K440, KM540 to K540, D156 to RGB10, D154 to RGB8, D155 to RGB9
Connections:
- net Col3: now also DK34.2 (A); no longer K340.1, K341.1
- net Col4: now also DK44.2 (A); no longer K440.1
- net Col5: now also DK54.2 (A); no longer K540.1, K541.1
- net Row4: now also K340.2, K341.2, K440.2, K540.2, K541.2; no longer DK34.1 (K), DK44.1 (K), DK54.1 (K)
- new net: DK34.1 (K), K340.1, K341.1
- new net: DK44.1 (K), K440.1
- new net: DK54.1 (K), K540.1, K541.1
Changed lines of the file:
@@
 $EndDescr
 $Comp
-L KEYSW KM340
+L KEYSW K340
 U 1 1 593C12F1
-P 5550 1250
-F 0 "KM340" H 5500 1250 60  0000 C CNN
-F 1 "LMB" H 5550 1150 60  0001 C CNN
-F 2 "Footprint:Mx_100" H 5550 1250 60  0001 C CNN
-F 3 "" H 5550 1250 60  0000 C CNN
-	1    5550 1250
-	1    0    0    -1
-$EndComp
-$Comp
-L KEYSW KM440
+P 5550 1300
+F 0 "K340" H 5500 1300 60  0001 C CNN
+F 1 "LMB" H 5550 1200 60  0000 C CNN
+F 2 "Footprint:Mx_100" H 5550 1300 60  0001 C CNN
+F 3 "" H 5550 1300 60  0000 C CNN
+	1    5550 1300
+	1    0    0    -1
+$EndComp
+$Comp
+L KEYSW K440
 U 1 1 593C13CC
-P 6400 1250
-F 0 "KM440" H 6350 1250 60  0000 C CNN
-F 1 "MMB" H 6400 1150 60  0001 C CNN
-F 2 "Footprint:Mx_100" H 6400 1250 60  0001 C CNN
-F 3 "" H 6400 1250 60  0000 C CNN
-	1    6400 1250
-	1    0    0    -1
-$EndComp
-$Comp
-L KEYSW KM540
+P 6400 1300
+F 0 "K440" H 6350 1300 60  0001 C CNN
+F 1 "MMB" H 6400 1200 60  0000 C CNN
+F 2 "Footprint:Mx_100" H 6400 1300 60  0001 C CNN
+F 3 "" H 6400 1300 60  0000 C CNN
+	1    6400 1300
+	1    0    0    -1
+$EndComp
+$Comp
+L KEYSW K540
 U 1 1 593C141B
-P 7250 1250
-F 0 "KM540" H 7200 1250 60  0000 C CNN
-F 1 "RMB" H 7250 1150 60  0001 C CNN
-F 2 "Footprint:Mx_100" H 7250 1250 60  0001 C CNN
-F 3 "" H 7250 1250 60  0000 C CNN
-	1    7250 1250
-	1    0    0    -1
-$EndComp
-$Comp
-L KEYSW KM341
+P 7250 1300
+F 0 "K540" H 7200 1300 60  0001 C CNN
+F 1 "RMB" H 7250 1200 60  0000 C CNN
+F 2 "Footprint:Mx_100" H 7250 1300 60  0001 C CNN
+F 3 "" H 7250 1300 60  0000 C CNN
+	1    7250 1300
+	1    0    0    -1
+$EndComp
+$Comp
+L KEYSW K341
 U 1 1 593C146D
-P 5550 1500
-F 0 "KM341" H 5500 1500 60  0000 C CNN
-F 1 "KEYSW" H 5550 1400 60  0001 C CNN
-F 2 "Footprint:Mx_125" H 5550 1500 60  0001 C CNN
-F 3 "" H 5550 1500 60  0000 C CNN
-	1    5550 1500
-	1    0    0    -1
-$EndComp
-$Comp
-L KEYSW KM541
+P 5550 1550
+F 0 "K341" H 5500 1550 60  0001 C CNN
+F 1 "LMB" H 5550 1450 60  0001 C CNN
+F 2 "Footprint:Mx_125" H 5550 1550 60  0001 C CNN
+F 3 "" H 5550 1550 60  0000 C CNN
+	1    5550 1550
+	1    0    0    -1
+$EndComp
+$Comp
+L KEYSW K541
 U 1 1 593C149E
-P 7250 1500
-F 0 "KM541" H 7200 1500 60  0000 C CNN
-F 1 "KEYSW" H 7250 1400 60  0001 C CNN
-F 2 "Footprint:Mx_125" H 7250 1500 60  0001 C CNN
-F 3 "" H 7250 1500 60  0000 C CNN
-	1    7250 1500
-	1    0    0    -1
-$EndComp
-$Comp
-L D DM34
+P 7250 1550
+F 0 "K541" H 7200 1550 60  0001 C CNN
+F 1 "RMB" H 7250 1450 60  0001 C CNN
+F 2 "Footprint:Mx_125" H 7250 1550 60  0001 C CNN
+F 3 "" H 7250 1550 60  0000 C CNN
+	1    7250 1550
+	1    0    0    -1
+$EndComp
+$Comp
+L D DK34
 U 1 1 593C18C0
-P 5250 1750
-F 0 "DM34" H 5250 1850 50  0000 C CNN
-F 1 "D" H 5250 1650 50  0000 C CNN
-F 2 "Footprint:D_SOD123" H 5250 1750 50  0001 C CNN
-F 3 "" H 5250 1750 50  0000 C CNN
-	1    5250 1750
+P 5850 1150
+F 0 "DK34" H 5850 1250 50  0001 C CNN
+F 1 "D43" H 5850 1050 50  0001 C CNN
+F 2 "Footprint:D_SOD123" H 5850 1150 50  0001 C CNN
+F 3 "" H 5850 1150 50  0000 C CNN
+	1    5850 1150
 	0    -1   -1   0
 $EndComp
 $Comp
-L D DM44
+L D DK44
 U 1 1 593C199F
-P 6100 1750
-F 0 "DM44" H 6100 1850 50  0000 C CNN
-F 1 "D" H 6100 1650 50  0000 C CNN
-F 2 "Footprint:D_SOD123" H 6100 1750 50  0001 C CNN
-F 3 "" H 6100 1750 50  0000 C CNN
-	1    6100 1750
+P 6700 1150
+F 0 "DK44" H 6700 1250 50  0001 C CNN
+F 1 "D44" H 6700 1050 50  0001 C CNN
+F 2 "Footprint:D_SOD123" H 6700 1150 50  0001 C CNN
+F 3 "" H 6700 1150 50  0000 C CNN
+	1    6700 1150
 	0    -1   -1   0
 $EndComp
 $Comp
-L D DM54
+L D DK54
 U 1 1 593C19F1
-P 6950 1750
-F 0 "DM54" H 6950 1850 50  0000 C CNN
-F 1 "D" H 6950 1650 50  0000 C CNN
-F 2 "Footprint:D_SOD123" H 6950 1750 50  0001 C CNN
-F 3 "" H 6950 1750 50  0000 C CNN
-	1    6950 1750
+P 7550 1150
+F 0 "DK54" H 7550 1250 50  0001 C CNN
+F 1 "D45" H 7550 1050 50  0001 C CNN
+F 2 "Footprint:D_SOD123" H 7550 1150 50  0001 C CNN
+F 3 "" H 7550 1150 50  0000 C CNN
+	1    7550 1150
 	0    -1   -1   0
 $EndComp
@@
 VCC
 Wire Wire Line
-	5850 1000 5850 1500
-Connection ~ 5850 1250
-Wire Wire Line
-	7550 1000 7550 1500
-Connection ~ 7550 1250
-Wire Wire Line
-	5250 1250 5250 1600
-Wire Wire Line
-	6950 1250 6950 1600
-Wire Wire Line
-	4750 1900 6950 1900
+	6950 1900 4750 1900
 Connection ~ 6100 1900
 Connection ~ 5250 1900
-Connection ~ 5250 1500
-Wire Wire Line
-	6100 1250 6100 1600
-Connection ~ 6950 1500
 Wire Wire Line
 	2350 1600 2500 1600
@@
 Text Label 1350 800  0    60   ~ 0
 Col5
-Text Label 7550 1000 0    60   ~ 0
+Text Label 7600 900  0    60   ~ 0
 Col5
 Text Label 8050 1250 0    60   ~ 0
@@
 Wire Wire Line
 	8050 1250 8300 1250
-Text Label 6700 1000 0    60   ~ 0
+Text Label 6750 900  0    60   ~ 0
 Col4
 Text Label 1350 1050 0    60   ~ 0
@@
 Text Label 8050 1150 0    60   ~ 0
 Col3
-Text Label 5850 1000 0    60   ~ 0
+Text Label 5900 900  0    60   ~ 0
 Col3
 Wire Wire Line
@@
 Text Label 8050 1050 0    60   ~ 0
 VCC
-Text Notes 4850 850  0    60   ~ 0
+Text Notes 4800 850  0    60   ~ 0
 Buttons
-Wire Wire Line
-	6700 1000 6700 1250
 Wire Notes Line
 	4650 700  7850 700
@@
 	1700 2100 1700 700
 $Comp
-L WS2812B D154
+L WS2812B RGB8
 U 1 1 593D8D65
 P 2000 2750
-F 0 "D154" H 1850 2950 50  0000 L CNN
-F 1 "WS2812B" H 1800 2550 50  0000 L CNN
+F 0 "RGB8" H 1850 2950 50  0000 L CNN
+F 1 "WS2812B" H 1800 2550 50  0001 L CNN
 F 2 "Footprint:WS2812B" H 2000 2750 50  0001 L CNN
 F 3 "" H 2000 2750 60  0000 C CNN
@@
 $EndComp
 $Comp
-L WS2812B D155
+L WS2812B RGB9
 U 1 1 593D8DC9
 P 2000 3350
-F 0 "D155" H 1850 3550 50  0000 L CNN
-F 1 "WS2812B" H 1800 3150 50  0000 L CNN
+F 0 "RGB9" H 1850 3550 50  0000 L CNN
+F 1 "WS2812B" H 1800 3150 50  0001 L CNN
 F 2 "Footprint:WS2812B" H 2000 3350 50  0001 L CNN
 F 3 "" H 2000 3350 60  0000 C CNN
@@
 $EndComp
 $Comp
-L WS2812B D156
+L WS2812B RGB10
 U 1 1 593D8E2F
 P 2000 3950
-F 0 "D156" H 1850 4150 50  0000 L CNN
-F 1 "WS2812B" H 1800 3750 50  0000 L CNN
+F 0 "RGB10" H 1850 4150 50  0000 L CNN
+F 1 "WS2812B" H 1800 3750 50  0001 L CNN
 F 2 "Footprint:WS2812B" H 2000 3950 50  0001 L CNN
 F 3 "" H 2000 3950 60  0000 C CNN
@@
 	1650 3450 1650 3650
 $Comp
-L C C17
+L C CRGB8
 U 1 1 593DAB4F
 P 1300 2800
-F 0 "C17" H 1325 2900 50  0000 L CNN
+F 0 "CRGB8" H 1325 2900 50  0001 L CNN
 F 1 "0.1u" H 1325 2700 50  0000 L CNN
 F 2 "Capacitors_SMD:C_0805_HandSoldering" H 1338 2650 50  0001 C CNN
@@
 Connection ~ 1000 3250
 $Comp
-L C C18
+L C CRGB9
 U 1 1 593DB8F3
 P 1300 3400
-F 0 "C18" H 1325 3500 50  0000 L CNN
+F 0 "CRGB9" H 1325 3500 50  0001 L CNN
 F 1 "0.1u" H 1325 3300 50  0000 L CNN
 F 2 "Capacitors_SMD:C_0805_HandSoldering" H 1338 3250 50  0001 C CNN
@@
 $EndComp
 $Comp
-L C C19
+L C CRGB10
 U 1 1 593DB954
 P 1300 4000
-F 0 "C19" H 1325 4100 50  0000 L CNN
+F 0 "CRGB10" H 1325 4100 50  0001 L CNN
 F 1 "0.1u" H 1325 3900 50  0000 L CNN
 F 2 "Capacitors_SMD:C_0805_HandSoldering" H 1338 3850 50  0001 C CNN
@@
 Connection ~ 1300 3250
 Connection ~ 1300 3850
+Wire Wire Line
+	5850 1300 5850 1550
+Wire Wire Line
+	5250 1300 5250 1900
+Wire Wire Line
+	5900 900  5850 900
+Wire Wire Line
+	5850 900  5850 1000
+Connection ~ 5250 1550
+Wire Wire Line
+	6750 900  6700 900
+Wire Wire Line
+	6700 900  6700 1000
+Wire Wire Line
+	6100 1300 6100 1900
+Wire Wire Line
+	7600 900  7550 900
+Wire Wire Line
+	7550 900  7550 1000
+Wire Wire Line
+	7550 1300 7550 1550
+Wire Wire Line
+	6950 1300 6950 1900
+Connection ~ 6950 1550
 $EndSCHEMATC

Commit message: - First commit for splitted spacebar
Parts:
- DK84: renamed from DK54; value D45 -> D48
- renumbered K540 to K840, K541 to K841
Connections:
- net Col5: no longer DK84.2 (A)
- new net Col8: DK84.2 (A)
Changed lines of the file:
@@
 $EndComp
 $Comp
-L KEYSW K540
+L KEYSW K840
 U 1 1 593C141B
 P 7250 1300
-F 0 "K540" H 7200 1300 60  0001 C CNN
+F 0 "K840" H 7200 1300 60  0001 C CNN
 F 1 "RMB" H 7250 1200 60  0000 C CNN
 F 2 "Footprint:Mx_100" H 7250 1300 60  0001 C CNN
@@
 $EndComp
 $Comp
-L KEYSW K541
+L KEYSW K841
 U 1 1 593C149E
 P 7250 1550
-F 0 "K541" H 7200 1550 60  0001 C CNN
+F 0 "K841" H 7200 1550 60  0001 C CNN
 F 1 "RMB" H 7250 1450 60  0001 C CNN
 F 2 "Footprint:Mx_125" H 7250 1550 60  0001 C CNN
@@
 $EndComp
 $Comp
-L D DK54
+L D DK84
 U 1 1 593C19F1
 P 7550 1150
-F 0 "DK54" H 7550 1250 50  0001 C CNN
-F 1 "D45" H 7550 1050 50  0001 C CNN
+F 0 "DK84" H 7550 1250 50  0001 C CNN
+F 1 "D48" H 7550 1050 50  0001 C CNN
 F 2 "Footprint:D_SOD123" H 7550 1150 50  0001 C CNN
 F 3 "" H 7550 1150 50  0000 C CNN
@@
 $EndComp
 Text HLabel 1100 800  0    60   Input ~ 0
-Col5
+Col8
 Text HLabel 1100 900  0    60   Input ~ 0
 Col4
@@
 D2
 Text Label 1350 800  0    60   ~ 0
-Col5
+Col8
 Text Label 7600 900  0    60   ~ 0
-Col5
+Col8
 Text Label 8050 1250 0    60   ~ 0
 Col5

Commit message: - Added Splitted spacebar
Connections:
- net Col5 is gone; now on net Col8: P2.5 (P5)
Changed lines of the file:
@@
 Col8
 Text Label 8050 1250 0    60   ~ 0
-Col5
+Col8
 Wire Wire Line
 	8050 1150 8300 1150

Commit message: Removed useless libraries
Merging all components in one library file to simplify maintenance
Parts:
- C9: manf# (none) -> CC1206ZKY5V9BB225
- CRGB10, CRGB8, CRGB9: manf# (none) -> CC0805ZRY5V9BB104
- K340, K341, K440, K840, K841: manf# (none) -> MX1A-C1NW
- P2: manf# (none) -> 53048-1010
- P3: manf# (none) -> 53048-0510
- R7, R8: manf# (none) -> CR0805-FX-4701ELF
- R9: manf# (none) -> RC0805FR-07100KL
- RGB10, RGB8, RGB9: manf# (none) -> COM-13667
Changed lines of the file:
@@
 EESchema Schematic File Version 2
-LIBS:74xgxx
-LIBS:74xx
-LIBS:ac-dc
-LIBS:actel
-LIBS:adc-dac
-LIBS:allegro
-LIBS:Altera
-LIBS:analog_devices
-LIBS:analog_switches
-LIBS:audio
-LIBS:battery_management
-LIBS:bbd
-LIBS:bosch
-LIBS:brooktre
-LIBS:cmos4000
-LIBS:cmos_ieee
-LIBS:conn
-LIBS:contrib
-LIBS:cypress
-LIBS:dc-dc
-LIBS:device
-LIBS:digital-audio
-LIBS:diode
-LIBS:display
-LIBS:dsp
-LIBS:elec-unifil
-LIBS:ESD_Protection
-LIBS:ftdi
-LIBS:gennum
-LIBS:graphic_symbols
-LIBS:hc11
-LIBS:infineon
-LIBS:intel
-LIBS:interface
-LIBS:intersil
-LIBS:ir
-LIBS:Lattice
-LIBS:leds
-LIBS:LEM
-LIBS:linear
-LIBS:logic_programmable
-LIBS:maxim
-LIBS:mechanical
-LIBS:memory
-LIBS:microchip
-LIBS:microchip_dspic33dsc
-LIBS:microchip_pic10mcu
-LIBS:microchip_pic12mcu
-LIBS:microchip_pic16mcu
-LIBS:microchip_pic18mcu
-LIBS:microchip_pic24mcu
-LIBS:microchip_pic32mcu
-LIBS:microcontrollers
-LIBS:modules
-LIBS:motor_drivers
-LIBS:motorola
-LIBS:motors
-LIBS:msp430
-LIBS:nordicsemi
-LIBS:nxp
-LIBS:nxp_armmcu
-LIBS:onsemi
-LIBS:opto
-LIBS:Oscillators
-LIBS:philips
-LIBS:power
-LIBS:powerint
-LIBS:Power_Management
-LIBS:pspice
-LIBS:references
-LIBS:regul
-LIBS:relays
-LIBS:rfcom
-LIBS:RFSolutions
-LIBS:sensors
-LIBS:silabs
-LIBS:siliconi
-LIBS:stm8
-LIBS:stm32
-LIBS:supertex
-LIBS:switches
-LIBS:texas
-LIBS:transf
-LIBS:transistors
-LIBS:triac_thyristor
-LIBS:ttl_ieee
-LIBS:valves
-LIBS:video
-LIBS:wiznet
-LIBS:Xicor
-LIBS:xilinx
-LIBS:zetex
-LIBS:Zilog
 LIBS:keyboard_parts
-LIBS:mkl27z256vfm4
-LIBS:Trackpad
-LIBS:TS65
 LIBS:DK60TP-cache
 EELAYER 25 0
@@
 encoding utf-8
 Sheet 4 7
-Title ""
-Date ""
-Rev ""
-Comp ""
+Title "DK60TP"
+Date "2017-10-14"
+Rev "B"
+Comp "DarKou.fr"
 Comment1 ""
 Comment2 ""
@@
 F 1 "LMB" H 5550 1200 60  0000 C CNN
 F 2 "Footprint:Mx_100" H 5550 1300 60  0001 C CNN
-F 3 "" H 5550 1300 60  0000 C CNN
+F 3 "http://www.mouser.com/ds/2/71/mx_cat-526196.pdf" H 5550 1300 60  0001 C CNN
+F 4 "MX1A-C1NW" H 5550 1300 60  0001 C CNN "manf#"
 	1    5550 1300
 	1    0    0    -1
@@
 F 1 "MMB" H 6400 1200 60  0000 C CNN
 F 2 "Footprint:Mx_100" H 6400 1300 60  0001 C CNN
-F 3 "" H 6400 1300 60  0000 C CNN
+F 3 "http://www.mouser.com/ds/2/71/mx_cat-526196.pdf" H 6400 1300 60  0001 C CNN
+F 4 "MX1A-C1NW" H 6400 1300 60  0001 C CNN "manf#"
 	1    6400 1300
 	1    0    0    -1
@@
 F 1 "RMB" H 7250 1200 60  0000 C CNN
 F 2 "Footprint:Mx_100" H 7250 1300 60  0001 C CNN
-F 3 "" H 7250 1300 60  0000 C CNN
+F 3 "http://www.mouser.com/ds/2/71/mx_cat-526196.pdf" H 7250 1300 60  0001 C CNN
+F 4 "MX1A-C1NW" H 7250 1300 60  0001 C CNN "manf#"
 	1    7250 1300
 	1    0    0    -1
@@
 F 1 "LMB" H 5550 1450 60  0001 C CNN
 F 2 "Footprint:Mx_125" H 5550 1550 60  0001 C CNN
-F 3 "" H 5550 1550 60  0000 C CNN
+F 3 "http://www.mouser.com/ds/2/71/mx_cat-526196.pdf" H 5550 1550 60  0001 C CNN
+F 4 "MX1A-C1NW" H 5550 1550 60  0001 C CNN "manf#"
 	1    5550 1550
 	1    0    0    -1
@@
 F 1 "RMB" H 7250 1450 60  0001 C CNN
 F 2 "Footprint:Mx_125" H 7250 1550 60  0001 C CNN
-F 3 "" H 7250 1550 60  0000 C CNN
+F 3 "http://www.mouser.com/ds/2/71/mx_cat-526196.pdf" H 7250 1550 60  0001 C CNN
+F 4 "MX1A-C1NW" H 7250 1550 60  0001 C CNN "manf#"
 	1    7250 1550
 	1    0    0    -1
@@
 F 1 "4.7K" V 3150 1400 50  0000 C CNN
 F 2 "Resistors_SMD:R_0805_HandSoldering" V 3080 1400 50  0001 C CNN
-F 3 "" H 3150 1400 50  0001 C CNN
+F 3 "http://www.mouser.com/ds/2/54/chpreztr-977002.pdf" H 3150 1400 50  0001 C CNN
+F 4 "CR0805-FX-4701ELF" V 3150 1400 60  0001 C CNN "manf#"
 	1    3150 1400
 	0    1    1    0
@@
 F 1 "4.7K" V 2800 1200 50  0000 C CNN
 F 2 "Resistors_SMD:R_0805_HandSoldering" V 2730 1200 50  0001 C CNN
-F 3 "" H 2800 1200 50  0001 C CNN
+F 3 "http://www.mouser.com/ds/2/54/chpreztr-977002.pdf" H 2800 1200 50  0001 C CNN
+F 4 "CR0805-FX-4701ELF" V 2800 1200 60  0001 C CNN "manf#"
 	1    2800 1200
 	0    1    1    0
@@
 F 1 "2.2u" H 3460 1320 50  0000 L CNN
 F 2 "Capacitors_SMD:C_0805_HandSoldering" H 3450 1400 50  0001 C CNN
-F 3 "" H 3450 1400 50  0001 C CNN
+F 3 "http://www.mouser.com/ds/2/447/Yageo_UPY-GP_NP0_16V-to-50V_9-358835.pdf" H 3450 1400 50  0001 C CNN
+F 4 "CC1206ZKY5V9BB225" H 3450 1400 60  0001 C CNN "manf#"
 	1    3450 1400
 	0    1    1    0
@@
 F 1 "100K" V 3800 1400 50  0000 C CNN
 F 2 "Resistors_SMD:R_0805_HandSoldering" V 3730 1400 50  0001 C CNN
-F 3 "" H 3800 1400 50  0001 C CNN
+F 3 "http://www.mouser.com/ds/2/447/Yageo_08112016_RC0805-968729.pdf" H 3800 1400 50  0001 C CNN
+F 4 "RC0805FR-07100KL" V 3800 1400 60  0001 C CNN "manf#"
 	1    3800 1400
 	0    -1   -1   0
@@
 F 1 "TRACKPOINT" V 2250 1400 50  0000 C CNN
 F 2 "Connectors_Molex:Molex_PicoBlade_53048-0510_05x1.25mm_Angled" H 2150 1400 50  0001 C CNN
-F 3 "" H 2150 1400 50  0000 C CNN
+F 3 "http://www.mouser.com/ds/2/276/0530480510_PCB_HEADERS-170992.pdf" H 2150 1400 50  0001 C CNN
+F 4 "53048-0510" H 2150 1400 60  0001 C CNN "manf#"
 	1    2150 1400
 	-1   0    0    1
@@
 F 1 "MAIN_BOARD" H 8550 950 50  0000 C CNN
 F 2 "Connectors_Molex:Molex_PicoBlade_53048-1010_10x1.25mm_Angled" H 8550 50  50  0001 C CNN
-F 3 "" H 8550 50  50  0000 C CNN
+F 3 "http://www.mouser.com/ds/2/276/0530481010_PCB_HEADERS-146506.pdf" H 8550 50  50  0001 C CNN
+F 4 "53048-1010" H 8550 1250 60  0001 C CNN "manf#"
 	1    8550 1250
 	1    0    0    -1
@@
 F 2 "Footprint:WS2812B" H 2000 2750 50  0001 L CNN
 F 3 "" H 2000 2750 60  0000 C CNN
+F 4 "COM-13667" H 2000 2750 60  0001 C CNN "manf#"
 	1    2000 2750
 	1    0    0    -1
@@
 F 2 "Footprint:WS2812B" H 2000 3350 50  0001 L CNN
 F 3 "" H 2000 3350 60  0000 C CNN
+F 4 "COM-13667" H 2000 3350 60  0001 C CNN "manf#"
 	1    2000 3350
 	1    0    0    -1
@@
 F 2 "Footprint:WS2812B" H 2000 3950 50  0001 L CNN
 F 3 "" H 2000 3950 60  0000 C CNN
+F 4 "COM-13667" H 2000 3950 60  0001 C CNN "manf#"
 	1    2000 3950
 	1    0    0    -1
@@
 Wire Wire Line
 	2350 3850 2250 3850
-Text Label 2650 4350 0    60   ~ 0
+Text Label 2650 4450 0    60   ~ 0
 GND
 Wire Wire Line
 	2250 4050 2650 4050
 Wire Wire Line
-	2650 2850 2650 4350
+	2650 2850 2650 4450
 Wire Wire Line
 	2250 3450 2650 3450
@@
 F 1 "0.1u" H 1325 2700 50  0000 L CNN
 F 2 "Capacitors_SMD:C_0805_HandSoldering" H 1338 2650 50  0001 C CNN
-F 3 "" H 1300 2800 50  0000 C CNN
+F 3 "http://www.yageo.com/documents/recent/UPY-GPHC_Y5V_6.3V-to-50V_8.pdf" H 1300 2800 50  0001 C CNN
+F 4 "CC0805ZRY5V9BB104" H 1300 2800 60  0001 C CNN "manf#"
 	1    1300 2800
 	1    0    0    -1
@@
 F 1 "0.1u" H 1325 3300 50  0000 L CNN
 F 2 "Capacitors_SMD:C_0805_HandSoldering" H 1338 3250 50  0001 C CNN
-F 3 "" H 1300 3400 50  0000 C CNN
+F 3 "http://www.yageo.com/documents/recent/UPY-GPHC_Y5V_6.3V-to-50V_8.pdf" H 1300 3400 50  0001 C CNN
+F 4 "CC0805ZRY5V9BB104" H 1300 3400 60  0001 C CNN "manf#"
 	1    1300 3400
 	1    0    0    -1
@@
 F 1 "0.1u" H 1325 3900 50  0000 L CNN
 F 2 "Capacitors_SMD:C_0805_HandSoldering" H 1338 3850 50  0001 C CNN
-F 3 "" H 1300 4000 50  0000 C CNN
+F 3 "http://www.yageo.com/documents/recent/UPY-GPHC_Y5V_6.3V-to-50V_8.pdf" H 1300 4000 50  0001 C CNN
+F 4 "CC0805ZRY5V9BB104" H 1300 4000 60  0001 C CNN "manf#"
 	1    1300 4000
 	1    0    0    -1
