File: Kicad/DK60TP.kicad_pcb (KiCad board)
At the start: 2 copper layers, 285 x 113.5 mm, 322 parts, among them J1 USB_mini_micro_B, J2 RGB, J3 CAPS_LOCK, K0 K00, K10 K10, K100 K01, K110 K11, K120 K21, K130 K31, K140 K41, K141 K41, K20 K20, K200 K02, K21 K20, K210 K12, K220 K22, K230 K32, K240 K42, K241 K42, K30 K30, K300 K03, K31 K30, K310 K13, K320 K23, K330 K33, K340 LMB, K341 LMB, K40 K40, K400 K04, K41 K40, K410 K14, K420 K24, K430 K34, K440 MMB, K4C1 K4C, K500 K05, K510 K15, K520 K25, K530 K35, K540 RMB, K541 RMB, K600 K06, K610 K16, K620 K26, K630 K36, K640 K46, K641 K46, K642 K46, K700 K07, K710 K17, K720 K27, K730 K37, K800 K08, K810 K18, K820 K28, K830 K38, K900 K09, K910 K19, K920 K29, K930 K39, K940 K49, M1 MISC, M2 MISC, P1 MOUSE_BOARD, P2 MAIN_BOARD, P3 TRACKPOINT, SW1 SW_PUSH, U0 ATMEGA32U4-MU, U1 PAM2804, X1 XTAL_GND

Commit message: - Added Splitted spacebar
Parts:
- removed K541: RMB, Footprint:Mx_125
- added DK74: D47, Footprint:D_SOD123, B.Cu at (225.2, 118.1)
- added DK84: D48, Footprint:D_SOD123, B.Cu at (207.4, 137.9)
- added K643: K46, Footprint:Mx_100, F.Cu at (201.5, 125.2)
- added K740: K47, Footprint:Mx_225, F.Cu at (232.5, 125.2)
- added K840: RMB, Footprint:Mx_100, F.Cu at (211.0, 144.2)
- added K841: RMB, Footprint:Mx_125, F.Cu at (213.4, 144.2)
- added SPC_225_0: SPC_225_0, Footprint:MXST, F.Cu at (220.6, 125.2)
- added SPC_275_0: SPC_275_0, Footprint:MXST, F.Cu at (153.9, 125.2)
- added SPC_275_1: SPC_275_1, Footprint:MXST, F.Cu at (177.7, 125.2)
- K540: value RMB -> K465; footprint Footprint:Mx_100 -> Footprint:Mx_275
- moved DK54 50.9 mm to (158.2, 124.9), turned to 270 degrees
- moved K540 49.1 mm to (165.8, 125.2)
- moved X1 27.0 mm to (147.8, 127.2)
- moved C2 24.8 mm to (152.8, 129.1), turned to 0 degrees
- moved C1 23.1 mm to (153.4, 127.1), turned to 0 degrees
- moved U0 20.5 mm to (139.5, 124.2), turned to 225 degrees
- moved C4 19.6 mm to (130.6, 129.7)
- moved R2 18.2 mm to (131.6, 131.7)
- moved C6 16.3 mm to (150.6, 120.5)
- moved C7 16.1 mm to (131.6, 117.6), turned to 180 degrees
- moved C8 16.0 mm to (144.3, 113.3), turned to 0 degrees
- moved C3 15.6 mm to (137.8, 116.6)
- moved C5 13.2 mm to (154.8, 125.1)
- moved J3 12.3 mm to (223.8, 111.1), turned to 90 degrees
- moved P1 6.42 mm to (216.8, 126.1)
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Connections:
- DK54 pad 2: /TRACKPOINT/Col5 -> Col5
- J1 pad 4: Net-(J1-Pad4) -> (no net)
- K540 pad 2: /TRACKPOINT/Row4 -> Row4
- K642 pad 1: Net-(DK64-Pad1) -> Row4
- K642 pad 2: Row4 -> Net-(DK64-Pad1)
- MH2 pad 1: Net-(MH2-Pad1) -> (no net)
- MH7 pad 1: Net-(MH7-Pad1) -> (no net)
- P1 pad 5: Col5 -> Col8
- P1 pad 9: Net-(P1-Pad9) -> (no net)
- P2 pad 5: /TRACKPOINT/Col5 -> /TRACKPOINT/Col8
- P2 pad 9: Net-(P2-Pad9) -> (no net)
- RGB10 pad 2: Net-(RGB10-Pad2) -> (no net)
- U0 pad 26: Col8 -> Row4
- U0 pad 28: Col9 -> Col0
- U0 pad 29: Row2 -> Col1
- U0 pad 30: Col4 -> Row2
- U0 pad 31: Row1 -> Col2
- U0 pad 32: Row4 -> Row0
- U0 pad 36: Col0 -> Col3
- U0 pad 37: Row0 -> Col4
- U0 pad 38: Col1 -> Row1
- U0 pad 39: Col2 -> Col8
- U0 pad 40: Col3 -> Col9
- U0 pad 41: Net-(U0-Pad41) -> (no net)
- U0 pad 42: Net-(U0-Pad42) -> (no net)
Routing:
- net Col8: track 149.7 -> 244.0 mm, vias 4 -> 6
- net /TRACKPOINT/Col8: track 0.00 -> 84.4 mm
- net /TRACKPOINT/Col5: track 84.4 -> 0.00 mm
- net Col7: track 127.1 -> 191.6 mm, vias 2 -> 4
- net VCC: track 1061.4 -> 1114.2 mm, vias 20 -> 22
- net Col4: track 188.0 -> 237.4 mm, vias 6 -> 4
- net Col9: track 288.7 -> 325.9 mm, vias 4 -> 6
- net ColA: track 184.4 -> 217.0 mm
- net BACKLIT: track 92.0 -> 124.3 mm, vias 2 -> 4
- net RGB: track 53.1 -> 85.2 mm, vias 0 -> 2
- net Row2: track 368.1 -> 341.0 mm, vias 2 -> 0
- net ColD: track 280.9 -> 306.9 mm
- net D2: track 64.5 -> 89.4 mm
- net Net-(J3-Pad2): track 204.6 -> 182.1 mm
- net D5: track 65.1 -> 86.9 mm, vias 3 -> 5
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
Commit message: - Routing and moved components near holes
Parts:
- added BL540: LED, Footprint:LED_TH_BIVAR, F.Cu at (165.8, 130.2)
- added BL740: LED, Footprint:LED_TH_BIVAR, F.Cu at (232.5, 130.2)
- K540: value K465 -> K45
- moved C11 36.9 mm to (279.6, 109.7), turned to 270 degrees
- moved L1 26.1 mm to (275.8, 112.9)
- moved U1 4.77 mm to (249.8, 115.5)
- moved R5 4.65 mm to (249.0, 121.7)
- moved DKD2 2.40 mm to (323.2, 78.9), turned to 90 degrees
- moved DK74 1.20 mm to (225.2, 119.3)
- moved P1 0.21 mm to (217.0, 126.1)
- turned BLD20 to 180 degrees
Routing:
- net GND: track 1095.5 -> 1441.7 mm, vias 14 -> 18
- net VCC: track 1114.2 -> 1254.0 mm, vias 22 -> 21
- net LED_AN: track 1605.3 -> 1638.9 mm, vias 1 -> 3
- net Net-(L1-Pad1): track 3.51 -> 33.5 mm, vias 0 -> 2
- net LED_CATH: track 1575.4 -> 1598.9 mm
- net RGB: track 85.2 -> 76.3 mm
- net Col7: track 191.6 -> 200.3 mm
- net Row4: track 402.3 -> 408.6 mm, vias 4 -> 1
- net Col5: track 172.4 -> 166.2 mm
- net D5: track 86.9 -> 92.7 mm, vias 5 -> 1
- net ColD: track 306.9 -> 301.4 mm
- net Net-(RGB6-Pad2): track 70.4 -> 75.9 mm
- net Row1: track 373.7 -> 378.2 mm
- net D2: track 89.4 -> 85.4 mm
- net Col3: track 240.6 -> 237.5 mm
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
Commit message: Removed values/references on PCB
Parts:
- P1: value MOUSE_BOARD -> TRACKPOINT
- moved MH9 55.6 mm to (286.2, 114.7)
- moved R5 43.4 mm to (292.0, 116.1), turned to 180 degrees
- moved C10 31.5 mm to (286.0, 114.7), turned to 180 degrees
- moved U1 31.0 mm to (280.8, 115.5)
- moved C11 6.39 mm to (277.4, 103.7)
- moved L1 3.85 mm to (277.6, 109.5), turned to 180 degrees
- moved DK83 2.82 mm to (228.2, 99.5), turned to 0 degrees
- moved J2 2.01 mm to (245.6, 124.1), turned to 90 degrees
- moved DK64 1.16 mm to (182.6, 119.9)
- moved DK54 0.46 mm to (158.6, 125.1)
- renumbered SW1 to RESET
Routing:
- net GND: track 1441.7 -> 1561.0 mm, vias 18 -> 16
- net Net-(L1-Pad1): track 33.5 -> 5.29 mm, vias 2 -> 0
- net BACKLIT: track 126.4 -> 149.3 mm
- net VCC: track 1254.0 -> 1233.9 mm, vias 21 -> 22
- net DOUT: track 127.5 -> 116.0 mm, vias 2 -> 1
- net LED_CATH: track 1598.9 -> 1589.2 mm, vias 9 -> 7
- net Row4: track 408.6 -> 415.8 mm
- net LED_AN: track 1638.9 -> 1644.0 mm
- net Col8: track 242.1 -> 237.6 mm
- net Net-(RGB2-Pad2): track 63.5 -> 66.1 mm
- net Row3: track 302.9 -> 304.7 mm
- net Net-(DK64-Pad1): track 44.6 -> 43.4 mm
- net Net-(DK83-Pad1): track 4.26 -> 5.35 mm
- net Col0: track 163.4 -> 162.6 mm
- net Col6: track 137.8 -> 138.5 mm
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
Commit message: Routing
Parts:
- moved DKB4 6.32 mm to (278.8, 124.1), turned to 270 degrees
- moved MH7 0.71 mm to (192.2, 95.9)
Routing:
- net LED_CATH: track 1589.2 -> 1612.9 mm
- net GND: track 1561.0 -> 1583.8 mm, vias 16 -> 19
- net ColB: track 232.0 -> 245.9 mm
- net Net-(DKD3-Pad1): track 19.3 -> 32.1 mm
- net Col4: track 236.1 -> 225.2 mm
- net VCC: track 1233.9 -> 1240.1 mm
- net Col9: track 325.7 -> 330.5 mm
- net LED_AN: track 1644.0 -> 1648.1 mm
- net Row4: track 415.8 -> 412.0 mm
- net Col3: track 237.5 -> 234.0 mm
- net ColA: track 215.0 -> 212.1 mm
- net BACKLIT: track 149.3 -> 146.9 mm
- net Col7: track 199.8 -> 197.8 mm
- net ColC: track 270.6 -> 272.5 mm
- net Net-(DKB4-Pad1): track 8.82 -> 10.4 mm
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
Commit message: Changed Crystal
Replaced crystal with 2 poles crystal
Parts:
- removed X1: XTAL_GND, Footprint:FA-238
- added Y1: Crystal, Crystals:Crystal_SMD_0603-2pin_6.0x3.5mm, B.Cu at (149.2, 126.9)
- P1: value TRACKPOINT -> MOUSE_BOARD
- SW1: renamed from RESET; value SW_PUSH -> RESET
- moved DK54 14.5 mm to (172.2, 120.1), turned to 90 degrees
- moved C6 3.60 mm to (147.0, 120.3)
- moved C1 2.78 mm to (154.8, 124.7)
- moved C5 2.55 mm to (156.6, 126.9), turned to 180 degrees
- moved C2 2.01 mm to (154.8, 129.1)
Routing:
- net Col5: track 166.2 -> 141.9 mm
- net GND: track 1583.8 -> 1560.9 mm
- net ColC: track 272.5 -> 267.8 mm
- net D5: track 92.7 -> 96.5 mm, vias 1 -> 3
- net Net-(DK54-Pad1): track 6.27 -> 9.35 mm, vias 1 -> 0
- net D2: track 85.4 -> 88.3 mm
- net RGB: track 76.3 -> 78.3 mm
- net XTAL2: track 10.9 -> 12.7 mm
- net XTAL1: track 11.7 -> 13.5 mm
- net Net-(R4-Pad1): track 33.2 -> 32.2 mm
- net ColB: track 245.9 -> 246.8 mm
- net Net-(R3-Pad1): track 30.2 -> 29.3 mm
- net /TRACKPOINT/RGB: track 187.3 -> 188.0 mm
- net VCC: track 1240.1 -> 1240.5 mm, vias 22 -> 24
- net RESET: track 158.3 -> 158.1 mm, vias 2 -> 4

Commit message: Routing / Filled zone
- Cleaning routing
- Increase filled zone for B layer
Parts:
- moved DK10 13.4 mm to (96.6, 54.1), turned to 270 degrees
- moved DKD3 3.12 mm to (327.0, 97.3)
- moved C7 2.38 mm to (129.6, 116.3)
- moved DK1 2.20 mm to (70.6, 61.5)
- moved DKC2 1.99 mm to (309.0, 80.7)
- moved R3 1.99 mm to (135.6, 92.9)
- moved DKD0 1.85 mm to (312.4, 51.9)
- moved DK22 1.39 mm to (119.2, 80.7)
- moved DK14 0.80 mm to (94.8, 119.7)
- moved C3 0.40 mm to (137.4, 116.7)
- moved KDC0 0.40 mm to (293.0, 51.9)
Routing:
- net GND: track 1560.9 -> 1307.8 mm, vias 19 -> 5
- net VCC: track 1240.5 -> 1228.5 mm
- net Col1: track 132.8 -> 121.1 mm
- net BACKLIT: track 147.2 -> 155.6 mm
- net Net-(DK10-Pad1): track 4.20 -> 12.4 mm
- net /TRACKPOINT/Col8: track 84.4 -> 92.4 mm
- net /TRACKPOINT/Col4: track 65.8 -> 73.5 mm
- net Row3: track 304.7 -> 311.9 mm
- net ColD: track 301.5 -> 294.7 mm
- net D2: track 88.3 -> 95.0 mm
- net Col9: track 330.5 -> 324.1 mm
- net LED_CATH: track 1612.9 -> 1607.1 mm
- net RGB: track 78.3 -> 72.6 mm
- net ColA: track 212.3 -> 207.7 mm
- net Net-(DK64-Pad1): track 43.4 -> 47.8 mm
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
Commit message: - Increased GND area
Parts:
- moved C8 0.80 mm to (143.6, 112.9)
Connections:
- K21 pad 1: Net-(DK2-Pad1) -> Row2
- K21 pad 2: Row2 -> Net-(DK2-Pad1)
Routing:
- net LED_AN: track 1644.5 -> 1607.3 mm, vias 3 -> 11
- net Row0: track 423.0 -> 395.7 mm
- net Row2: track 343.4 -> 355.0 mm
- net GND: track 1307.8 -> 1314.9 mm, vias 5 -> 6
- net VCC: track 1228.5 -> 1233.9 mm
- net LED_CATH: track 1607.1 -> 1604.5 mm, vias 7 -> 6
- net Col9: track 324.1 -> 322.0 mm
- net Col2: track 113.7 -> 115.7 mm
- net RESET: track 159.0 -> 160.7 mm
- net ColC: track 271.3 -> 270.0 mm
- net Col0: track 162.9 -> 163.8 mm
- net Col1: track 121.1 -> 120.3 mm
- net Row4: track 409.7 -> 410.4 mm
- net Net-(C8-Pad1): track 10.8 -> 10.2 mm
- net RGB: track 72.6 -> 73.2 mm
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
Commit message: - Some changes (routing/ground area/space)
- Updated routing
- Increased ground area
- Invert Split space 2.75U/2.25U
- Added missing led for backlit
Parts:
- removed SPC_275_1: SPC_275_1, Footprint:MXST
- added BL643: LED, Footprint:LED_TH_BIVAR, F.Cu at (191.8, 130.2)
- added SPC_R_SPLIT_1: SPC_275_1, Footprint:MXST, F.Cu at (239.6, 125.2)
- K540: footprint Footprint:Mx_275 -> Footprint:Mx_225
- K740: footprint Footprint:Mx_225 -> Footprint:Mx_275
- SPC_R_SPLIT_0: renamed from SPC_225_0; value SPC_225_0 -> SPC_275_0
- moved SPC_275_0 19.1 mm to (173.0, 125.2)
- moved P1 12.9 mm to (211.6, 114.4), turned to 180 degrees
- moved DK54 11.3 mm to (161.4, 116.9), turned to 45 degrees
- moved K643 9.52 mm to (192.0, 125.2)
- moved DK64 5.22 mm to (178.0, 122.4)
- moved BL540 4.75 mm to (161.0, 130.2)
- moved K540 4.75 mm to (161.0, 125.2)
- moved BL740 4.75 mm to (227.7, 130.2)
- moved K740 4.75 mm to (227.7, 125.2)
- moved SPC_R_SPLIT_0 4.75 mm to (215.8, 125.2)
- moved C5 4.00 mm to (152.6, 126.9)
- moved C1 2.40 mm to (152.4, 124.7)
- moved C2 2.40 mm to (152.4, 129.1)
- moved CRGB6 2.13 mm to (324.8, 58.4)
- moved DK74 1.96 mm to (226.8, 118.2)
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Connections:
- K643 pad 1: Net-(DK64-Pad1) -> Row4
- K643 pad 2: Row4 -> Net-(DK64-Pad1)
Routing:
- net GND: track 1314.9 -> 885.2 mm, vias 6 -> 2
- net VCC: track 1233.9 -> 1169.4 mm, vias 24 -> 22
- net Col5: track 144.7 -> 113.3 mm
- net DOUT: track 116.0 -> 134.1 mm
- net Col8: track 239.5 -> 253.0 mm, vias 6 -> 8
- net Net-(DK64-Pad1): track 47.8 -> 37.7 mm, vias 0 -> 1
- net D5: track 94.2 -> 103.6 mm, vias 3 -> 2
- net LED_CATH: track 1604.5 -> 1611.2 mm
- net D2: track 95.0 -> 100.9 mm, vias 3 -> 2
- net ColB: track 248.0 -> 242.8 mm
- net Col0: track 163.8 -> 168.5 mm
- net Col6: track 140.7 -> 144.8 mm
- net Net-(DK54-Pad1): track 9.35 -> 5.82 mm
- net XTAL1: track 16.0 -> 12.6 mm
- net Col3: track 236.4 -> 233.0 mm
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Other:
- net class Backlit removed
