File: Kicad/DK60TP.kicad_pcb (KiCad board)
At the start: 2 copper layers, 285 x 113.5 mm, 333 parts, among them J1 USB_mini_micro_B, J2 RGB, J3 CAPS_LOCK, K0 K00, K10 K10, K100 K01, K110 K11, K120 K21, K130 K31, K140 K41, K141 K41, K20 K20, K200 K02, K21 K20, K210 K12, K220 K22, K230 K32, K240 K42, K241 K42, K30 K30, K300 K03, K31 K30, K310 K13, K320 K23, K330 K33, K340 LMB, K341 LMB, K40 K40, K400 K04, K41 K40, K410 K14, K420 K24, K430 K34, K440 MMB, K4C1 K4C, K500 K05, K510 K15, K520 K25, K530 K35, K540 K45, K600 K06, K610 K16, K620 K26, K630 K36, K640 K46, K641 K46, K642 K46, K643 K46, K700 K07, K710 K17, K720 K27, K730 K37, K740 K47, K800 K08, K810 K18, K820 K28, K830 K38, K840 RMB, K841 RMB, K900 K09, K910 K19, K920 K29, K930 K39, K940 K49, M1 MISC, M2 MISC, P1 MOUSE_BOARD, P2 MAIN_BOARD, P3 TRACKPOINT, SW1 RESET, U0 ATMEGA32U4-MU, U1 PAM2804, Y1 Crystal

Commit message: Fixed position of the USB port
Parts:
- moved J1 0.20 mm to (82.0, 44.0)
Changed lines of the file:
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@@
     (links 583)
     (no_connects 2)
-    (area 63.881249 39.906249 348.981251 153.506251)
+    (area 44.081251 23.35625 382.58125 192.356251)
     (thickness 1.6)
     (drawings 55)
-    (tracks 2668)
+    (tracks 2666)
     (zones 0)
     (modules 333)
@@
     (38 B.Mask user)
     (39 F.Mask user)
-    (40 Dwgs.User user)
+    (40 Dwgs.User user hide)
     (41 Cmts.User user)
     (42 Eco1.User user)
@@
   )
   (module Footprint:Micro_USB_Hand (layer B.Cu)
-    (at 82.245 43.98125 180)
+    (at 82.045 43.98125 180)
     (fp_text reference J1 (at 0 -2.05 180) (layer B.SilkS)
       (effects (font (size 1 1) (thickness 0.15)) (justify mirror))
@@
   (segment (start 141.931517 126.560413) (end 142.627354 127.25625) (width 0.25) (layer B.Cu) (net 5) (status 10))
   (segment (start 141.909163 126.560413) (end 141.917913 126.560413) (width 0.25) (layer B.Cu) (net 5) (status 30))
+  (segment (start 80.694998 44.831248) (end 80.694998 44.031252) (width 0.25) (layer B.Cu) (net 6) (status 800000))
+  (segment (start 80.694998 44.031252) (end 80.745 43.98125) (width 0.25) (layer B.Cu) (net 6) (status C00000))
+  (segment (start 80.694998 45.38125) (end 80.694998 44.831248) (width 0.5) (layer B.Cu) (net 6))
+  (segment (start 80.694998 45.78125) (end 80.694998 45.38125) (width 0.75) (layer B.Cu) (net 6))
+  (segment (start 81.045 50.98125) (end 81.055048 50.98125) (width 0.75) (layer B.Cu) (net 6))
+  (segment (start 82.445 52.371202) (end 82.445 52.98125) (width 0.75) (layer B.Cu) (net 6))
+  (segment (start 81.055048 50.98125) (end 82.445 52.371202) (width 0.75) (layer B.Cu) (net 6))
+  (segment (start 80.694998 50.631248) (end 80.694998 45.78125) (width 0.75) (layer B.Cu) (net 6))
+  (segment (start 80.694998 45.78125) (end 80.694998 45.58125) (width 0.75) (layer B.Cu) (net 6))
+  (segment (start 81.045 50.98125) (end 80.694998 50.631248) (width 0.75) (layer B.Cu) (net 6))
+  (segment (start 80.745 43.98125) (end 80.745 44.48125) (width 0.25) (layer B.Cu) (net 6) (status C00000))
   (segment (start 80.078 59.80625) (end 81.22 59.80625) (width 0.25) (layer B.Cu) (net 6))
   (segment (start 81.22 59.80625) (end 83.045 57.98125) (width 0.25) (layer B.Cu) (net 6))
@@
   (segment (start 83.12 58.05625) (end 83.045 57.98125) (width 0.75) (layer F.Cu) (net 6))
   (via (at 83.045 57.98125) (size 0.6) (drill 0.4) (layers F.Cu B.Cu) (net 6))
-  (segment (start 82.445 52.58125) (end 80.829375 50.965625) (width 0.75) (layer B.Cu) (net 6))
-  (segment (start 80.845 46.18125) (end 80.829375 46.18125) (width 0.5) (layer B.Cu) (net 6))
-  (segment (start 80.845 44.98125) (end 80.945 44.88125) (width 0.5) (layer B.Cu) (net 6))
-  (segment (start 80.829375 46.18125) (end 80.829375 50.965625) (width 0.75) (layer B.Cu) (net 6))
-  (segment (start 80.945 43.98125) (end 80.945 44.88125) (width 0.25) (layer B.Cu) (net 6))
-  (segment (start 80.845 44.98125) (end 80.845 46.18125) (width 0.5) (layer B.Cu) (net 6))
   (segment (start 83.045 57.98125) (end 82.445 57.38125) (width 0.75) (layer B.Cu) (net 6))
-  (segment (start 82.445 57.38125) (end 82.445 52.58125) (width 0.75) (layer B.Cu) (net 6))
-  (segment (start 80.945 43.18125) (end 80.945 43.08125) (width 0.5) (layer B.Cu) (net 6))
-  (segment (start 80.945 43.98125) (end 80.945 43.18125) (width 0.25) (layer B.Cu) (net 6))
-  (segment (start 80.945 43.08125) (end 81.045 42.98125) (width 0.25) (layer B.Cu) (net 6))
+  (segment (start 82.445 57.38125) (end 82.445 52.98125) (width 0.75) (layer B.Cu) (net 6))
   (segment (start 302.41375 108.85625) (end 302.41375 111.15) (width 0.25) (layer B.Cu) (net 6))
   (segment (start 308.77 117.50625) (end 319.005 117.50625) (width 0.25) (layer B.Cu) (net 6))
@@
   (segment (start 331.705 122.02) (end 331.08375 122.64125) (width 0.25) (layer B.Cu) (net 91) (status 30))
   (segment (start 331.08375 122.64125) (end 333.465 122.64125) (width 0.25) (layer B.Cu) (net 91) (status 30))
+  (segment (start 81.395 43.98125) (end 81.395 50.33125) (width 0.25) (layer B.Cu) (net 92) (status 400000))
+  (segment (start 81.395 50.33125) (end 82.045 50.98125) (width 0.25) (layer B.Cu) (net 92))
   (segment (start 125.445 60.38125) (end 127.81375 62.75) (width 0.25) (layer B.Cu) (net 92))
   (segment (start 127.81375 62.75) (end 127.81375 67.18125) (width 0.25) (layer B.Cu) (net 92))
@@
   (via (at 125.445 60.38125) (size 0.6) (drill 0.4) (layers F.Cu B.Cu) (net 92))
   (segment (start 125.045 59.98125) (end 125.445 60.38125) (width 0.25) (layer F.Cu) (net 92))
-  (segment (start 81.595 48.98125) (end 81.595 50.53125) (width 0.25) (layer B.Cu) (net 92))
-  (segment (start 81.595 50.53125) (end 91.045 59.98125) (width 0.25) (layer B.Cu) (net 92))
+  (segment (start 82.045 50.98125) (end 91.045 59.98125) (width 0.25) (layer B.Cu) (net 92))
   (via (at 92.445 59.98125) (size 0.6) (drill 0.4) (layers F.Cu B.Cu) (net 92))
   (segment (start 91.045 59.98125) (end 92.445 59.98125) (width 0.25) (layer B.Cu) (net 92))
-  (segment (start 81.595 47.18125) (end 81.595 48.98125) (width 0.25) (layer B.Cu) (net 92))
-  (segment (start 81.595 43.98125) (end 81.595 47.18125) (width 0.25) (layer B.Cu) (net 92))
+  (segment (start 82.045 43.98125) (end 82.045 50.18125) (width 0.25) (layer B.Cu) (net 93) (status 400000))
+  (segment (start 82.045 50.18125) (end 82.445 50.58125) (width 0.25) (layer B.Cu) (net 93))
   (segment (start 123.245 59.18125) (end 125.445 59.18125) (width 0.25) (layer F.Cu) (net 93))
   (segment (start 125.445 59.18125) (end 127.045 60.78125) (width 0.25) (layer F.Cu) (net 93))
-  (segment (start 82.23125 48.58125) (end 82.23125 50.3675) (width 0.25) (layer B.Cu) (net 93))
   (segment (start 123.045 59.18125) (end 123.245 59.18125) (width 0.25) (layer F.Cu) (net 93))
   (segment (start 109.445 59.18125) (end 123.045 59.18125) (width 0.25) (layer F.Cu) (net 93))
@@
   (via (at 93.245 59.18125) (size 0.6) (drill 0.4) (layers F.Cu B.Cu) (net 93))
   (segment (start 91.045 59.18125) (end 93.245 59.18125) (width 0.25) (layer B.Cu) (net 93))
-  (segment (start 82.23125 50.3675) (end 91.045 59.18125) (width 0.25) (layer B.Cu) (net 93))
+  (segment (start 82.445 50.58125) (end 91.045 59.18125) (width 0.25) (layer B.Cu) (net 93))
   (segment (start 128.263752 62.000002) (end 128.263752 62.78125) (width 0.25) (layer B.Cu) (net 93))
   (segment (start 127.045 60.78125) (end 128.263752 62.000002) (width 0.25) (layer B.Cu) (net 93))
@@
   (segment (start 128.263752 74.869854) (end 128.263752 62.78125) (width 0.25) (layer B.Cu) (net 93))
   (segment (start 135.109158 81.71526) (end 128.263752 74.869854) (width 0.25) (layer B.Cu) (net 93))
-  (segment (start 82.23125 47.58125) (end 82.23125 48.58125) (width 0.25) (layer B.Cu) (net 93))
-  (segment (start 82.23125 46.58125) (end 82.23125 43.995) (width 0.25) (layer B.Cu) (net 93))
-  (segment (start 82.23125 43.995) (end 82.245 43.98125) (width 0.25) (layer B.Cu) (net 93))
-  (segment (start 82.23125 47.58125) (end 82.23125 46.58125) (width 0.25) (layer B.Cu) (net 93))
   (segment (start 311.445 117.631252) (end 320.194998 117.631252) (width 0.25) (layer F.Cu) (net 94))
   (segment (start 322.578 115.24825) (end 322.578 114.35625) (width 0.25) (layer B.Cu) (net 94))

Commit message: - Increase GND area on Front layer
Routing:
- net LED_AN: track 1609.9 -> 1589.1 mm, vias 10 -> 12
- net Row4: track 411.3 -> 430.2 mm, vias 1 -> 2
- net VCC: track 1161.4 -> 1171.7 mm
- net Col9: track 322.0 -> 313.2 mm
- net Col3: track 233.0 -> 241.7 mm
- net Col4: track 222.9 -> 228.5 mm
- net CAPS_LED: track 90.9 -> 93.4 mm
- net DOUT: track 134.2 -> 136.1 mm, vias 1 -> 2
- net RESET: track 160.6 -> 158.9 mm
- net Row3: track 331.8 -> 332.9 mm
- net Col8: track 253.0 -> 254.0 mm
- net LED_CATH: track 1602.5 -> 1601.5 mm
- net Net-(RGB5-Pad2): track 65.9 -> 66.5 mm
- net ColD: track 294.3 -> 293.7 mm
- net Net-(RGB4-Pad2): track 73.4 -> 73.9 mm
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
Commit message: - Increased GND area on front layer
Parts:
- moved DK24 4.36 mm to (114.2, 118.8), turned to 90 degrees
Routing:
- net VCC: track 1171.7 -> 1162.9 mm, vias 22 -> 21
- net Col8: track 254.0 -> 258.7 mm, vias 8 -> 7
- net Net-(DK64-Pad1): track 38.2 -> 42.7 mm
- net ColA: track 207.9 -> 212.4 mm
- net Col9: track 313.2 -> 316.9 mm
- net D5: track 103.6 -> 106.9 mm
- net LED_AN: track 1589.1 -> 1586.0 mm, vias 12 -> 11
- net GND: track 587.9 -> 590.4 mm
- net D2: track 100.9 -> 103.3 mm
- net DOUT: track 136.1 -> 134.0 mm
- net RGB: track 75.4 -> 77.1 mm
- net ColC: track 271.4 -> 269.8 mm
- net Row2: track 356.4 -> 357.8 mm
- net CAPS_LED: track 93.4 -> 94.7 mm
- net Col6: track 144.8 -> 143.7 mm
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
Commit message: - Increased GND areas
Parts:
- turned BLD1 to 180 degrees
- turned BLD22 to 270 degrees
Routing:
- net LED_CATH: track 1600.5 -> 1576.2 mm, vias 8 -> 10
- net Row3: track 333.9 -> 341.4 mm
- net LED_AN: track 1586.0 -> 1593.5 mm
- net Col0: track 169.3 -> 172.5 mm
- net Net-(DK3-Pad1): track 14.3 -> 16.9 mm
- net Col4: track 228.5 -> 226.4 mm
- net Net-(DKD2-Pad1): track 30.2 -> 31.8 mm
- net VCC: track 1162.9 -> 1164.5 mm
- net BACKLIT: track 155.7 -> 154.6 mm, vias 4 -> 2
- net Col3: track 241.7 -> 240.7 mm
- net ColC: track 269.8 -> 269.0 mm
- net Col7: track 196.7 -> 196.0 mm
- net Row2: track 357.8 -> 358.5 mm
- net ColD: track 293.9 -> 293.3 mm
- net Col8: track 258.7 -> 258.4 mm, vias 7 -> 8

Commit message: - Fixed some bugs
* Fixed bug when trying to show 3D Viewer (bad egde cuts)
* Updated GND areas
* Fixed error when loading net list (bad chip name for holes)
Parts:
- moved DK34 8.59 mm to (159.6, 141.6)
- moved DK44 7.93 mm to (182.6, 143.4), turned to 270 degrees
- moved DK84 6.74 mm to (201.2, 140.6)
Routing:
- net GND: track 590.4 -> 71.7 mm
- net /TRACKPOINT/Col4: track 73.5 -> 59.2 mm
- net /TRACKPOINT/Col8: track 92.4 -> 81.5 mm
- net /TRACKPOINT/Col3: track 39.3 -> 31.0 mm
- net LED_AN: track 1593.5 -> 1601.1 mm, vias 11 -> 10
- net LED_CATH: track 1576.2 -> 1581.5 mm
- net Row2: track 358.5 -> 355.2 mm
- net Net-(RGB10-Pad4): track 98.8 -> 95.9 mm
- net VCC: track 1164.5 -> 1167.3 mm
- net Net-(DK34-Pad1): track 6.13 -> 7.86 mm
- net /TRACKPOINT/RGB: track 188.6 -> 187.4 mm
- net Net-(DK44-Pad1): track 4.53 -> 5.57 mm
- net Net-(DK84-Pad1): track 6.33 -> 7.13 mm
- net /TRACKPOINT/D2: track 156.3 -> 155.6 mm
- net /TRACKPOINT/D5: track 161.1 -> 160.5 mm
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Other:
- outline, holes or cut-outs redrawn

Commit message: - Added ivan ivanovitch layout
Parts:
- added 7U_LEFT_0: 7U_LEFT_0, Footprint:MXST, F.Cu at (130.1, 125.2)
- added K142: K41, Footprint:Mx_150, F.Cu at (106.3, 125.2)
- moved R2 7.11 mm to (138.6, 132.7)
- moved C7 5.27 mm to (131.7, 121.1), turned to 0 degrees
- moved C4 4.13 mm to (134.1, 131.8), turned to 270 degrees
- moved CRGB9 0.93 mm to (194.3, 151.0)
- moved DK14 0.68 mm to (94.7, 119.0)
- turned BLD31 to 180 degrees
Routing:
- net LED_AN: track 1601.1 -> 1566.6 mm, vias 10 -> 7
- net Net-(DK14-Pad1): track 6.49 -> 21.6 mm
- net BACKLIT: track 154.6 -> 146.0 mm
- net VCC: track 1167.3 -> 1160.0 mm
- net Net-(R2-Pad2): track 9.89 -> 16.0 mm
- net LED_CATH: track 1581.5 -> 1587.2 mm, vias 10 -> 9
- net GND: track 71.7 -> 67.1 mm
- net Row4: track 431.1 -> 435.4 mm
- net D5: track 106.9 -> 103.6 mm
- net Col2: track 116.1 -> 113.1 mm, vias 2 -> 4
- net Col8: track 258.4 -> 255.9 mm
- net /TRACKPOINT/Col8: track 81.5 -> 79.3 mm
- net ColB: track 243.2 -> 241.1 mm
- net Col1: track 120.5 -> 122.4 mm
- net ColD: track 293.3 -> 291.4 mm
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
Commit message: - Added missing led for ivan ivanovitch layout
Parts:
- added BL423: LED, Footprint:LED_TH_BIVAR, F.Cu at (106.3, 130.2)
Routing:
- net LED_CATH: track 1587.2 -> 1591.2 mm
- net LED_AN: track 1566.6 -> 1568.5 mm
Changed lines of the file:
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@@
 (kicad_pcb (version 4) (host pcbnew 4.0.7+dfsg1-1)
   (general
-    (links 585)
+    (links 587)
     (no_connects 2)
     (area 63.874999 39.891249 348.985001 153.511251)
     (thickness 1.6)
     (drawings 51)
-    (tracks 2772)
+    (tracks 2782)
     (zones 0)
-    (modules 335)
+    (modules 336)
     (nets 129)
   )
@@
     )
   )
+  (module Footprint:LED_TH_BIVAR (layer F.Cu)
+    (at 106.295 130.18125)
+    (descr "LED 3mm - Lead pitch 100mil (2,54mm)")
+    (tags "LED led 3mm 3MM 100mil 2,54mm")
+    (fp_text reference BL423 (at 0 -1.9) (layer F.SilkS)
+      (effects (font (size 0.8 0.8) (thickness 0.15)))
+    )
+    (fp_text value LED (at 0 2.032) (layer F.SilkS) hide
+      (effects (font (size 0.8 0.8) (thickness 0.15)))
+    )
+    (fp_text user + (at 3.048 0) (layer B.SilkS)
+      (effects (font (size 1 1) (thickness 0.15)) (justify mirror))
+    )
+    (pad 1 thru_hole rect (at -1.27 0) (size 1.7 1.7) (drill 1) (layers *.Cu *.Mask F.SilkS)
+      (net 1 LED_CATH))
+    (pad 2 thru_hole circle (at 1.27 0) (size 1.7 1.7) (drill 1) (layers *.Cu *.Mask F.SilkS)
+      (net 2 LED_AN))
+    (model ../../../../../home/dbroqua/Projects/dbroqua/DK60TP/Footprint/3D/LED-3MM.wrl
+      (at (xyz 0 0 0))
+      (scale (xyz 1 1 1))
+      (rotate (xyz 0 0 0))
+    )
+  )
   (gr_line (start 69.045 134.58125) (end 343.845 134.58125) (angle 90) (layer Edge.Cuts) (width 0.1))
   (gr_line (start 69.045 135.58125) (end 69.045 134.58125) (angle 90) (layer Edge.Cuts) (width 0.1))
@@
   (segment (start 123.345 113.65625) (end 123.345 113.78125) (width 0.25) (layer F.Cu) (net 0))
   (segment (start 123.345 113.78125) (end 123.345 113.65625) (width 0.25) (layer F.Cu) (net 0))
+  (segment (start 102.80125 130.18125) (end 105.025 130.18125) (width 0.25) (layer F.Cu) (net 1) (status C00000))
+  (segment (start 102.545 128.65625) (end 109.02 128.65625) (width 0.25) (layer F.Cu) (net 1))
+  (segment (start 109.045 128.68125) (end 109.045 130.18125) (width 0.25) (layer F.Cu) (net 1))
+  (segment (start 109.02 128.65625) (end 109.045 128.68125) (width 0.25) (layer F.Cu) (net 1))
   (segment (start 200.545 90.78125) (end 196.681398 90.78125) (width 0.25) (layer F.Cu) (net 1))
   (segment (start 196.531392 90.631244) (end 195.945 90.631244) (width 0.25) (layer F.Cu) (net 1))
@@
   (segment (start 102.745 128.65625) (end 102.745 130.125) (width 0.25) (layer F.Cu) (net 1))
   (segment (start 102.745 130.125) (end 102.80125 130.18125) (width 0.25) (layer F.Cu) (net 1))
-  (segment (start 102.80125 130.18125) (end 121.6925 130.18125) (width 0.25) (layer F.Cu) (net 1))
-  (segment (start 102.745 128.65625) (end 97.97 128.65625) (width 0.25) (layer F.Cu) (net 1))
+  (segment (start 109.045 130.18125) (end 121.6925 130.18125) (width 0.25) (layer F.Cu) (net 1))
+  (segment (start 102.745 128.65625) (end 102.545 128.65625) (width 0.25) (layer F.Cu) (net 1))
+  (segment (start 102.545 128.65625) (end 97.97 128.65625) (width 0.25) (layer F.Cu) (net 1))
   (segment (start 97.88 128.74625) (end 97.88 130.18125) (width 0.25) (layer F.Cu) (net 1))
   (segment (start 97.97 128.65625) (end 97.88 128.74625) (width 0.25) (layer F.Cu) (net 1))
@@
   (segment (start 74.0675 130.18125) (end 74.0675 129.79375) (width 0.25) (layer F.Cu) (net 1) (status 30))
   (segment (start 76.44875 73.03125) (end 76.44875 72.2125) (width 0.25) (layer F.Cu) (net 1) (status 30))
+  (segment (start 100.295 131.78125) (end 100.295 130.215) (width 0.25) (layer B.Cu) (net 2) (status 800000))
+  (segment (start 100.295 130.215) (end 100.26125 130.18125) (width 0.25) (layer B.Cu) (net 2) (status C00000))
+  (segment (start 99.545 131.78125) (end 100.295 131.78125) (width 0.25) (layer B.Cu) (net 2))
+  (segment (start 100.295 131.78125) (end 107.445 131.78125) (width 0.25) (layer B.Cu) (net 2))
+  (segment (start 107.565 131.66125) (end 107.565 130.18125) (width 0.25) (layer B.Cu) (net 2) (status 800000))
+  (segment (start 107.445 131.78125) (end 107.565 131.66125) (width 0.25) (layer B.Cu) (net 2))
+  (segment (start 107.545 131.85625) (end 107.545 130.20125) (width 0.25) (layer F.Cu) (net 2) (status 800000))
+  (segment (start 107.545 130.20125) (end 107.565 130.18125) (width 0.25) (layer F.Cu) (net 2) (status C00000))
   (segment (start 337.045 93.38125) (end 337.245 93.38125) (width 0.25) (layer F.Cu) (net 2))
   (segment (start 337.245 93.38125) (end 338.545 92.08125) (width 0.25) (layer F.Cu) (net 2))
@@
   (segment (start 332.57 112.65625) (end 333.7825 111.44375) (width 0.25) (layer F.Cu) (net 2))
   (segment (start 333.7825 111.44375) (end 333.7825 111.13125) (width 0.25) (layer F.Cu) (net 2))
-  (segment (start 100.445 131.85625) (end 100.445 130.20625) (width 0.25) (layer F.Cu) (net 2))
   (segment (start 100.445 130.20625) (end 100.42 130.18125) (width 0.25) (layer F.Cu) (net 2))
-  (segment (start 100.445 131.85625) (end 124.21375 131.85625) (width 0.25) (layer F.Cu) (net 2))
+  (segment (start 107.545 131.85625) (end 124.21375 131.85625) (width 0.25) (layer F.Cu) (net 2))
   (segment (start 124.21375 131.85625) (end 124.2325 131.8375) (width 0.25) (layer F.Cu) (net 2))
   (segment (start 124.2325 131.8375) (end 124.2325 130.18125) (width 0.25) (layer F.Cu) (net 2) (status 20))
@@
   (segment (start 84.91375 128.68125) (end 85.61375 127.98125) (width 0.25) (layer B.Cu) (net 2))
   (segment (start 76.6075 130.18125) (end 76.6075 131.44375) (width 0.25) (layer B.Cu) (net 2))
-  (segment (start 100.42 131.40625) (end 100.42 130.18125) (width 0.25) (layer B.Cu) (net 2))
-  (segment (start 100.045 131.78125) (end 100.42 131.40625) (width 0.25) (layer B.Cu) (net 2))
-  (segment (start 76.945 131.78125) (end 100.045 131.78125) (width 0.25) (layer B.Cu) (net 2))
+  (segment (start 76.945 131.78125) (end 99.545 131.78125) (width 0.25) (layer B.Cu) (net 2))
   (segment (start 76.6075 131.44375) (end 76.945 131.78125) (width 0.25) (layer B.Cu) (net 2))
   (segment (start 85.61375 127.98125) (end 85.61375 126.2125) (width 0.25) (layer F.Cu) (net 2))

Commit message: - Increased GND areas
Parts:
- moved C6 0.23 mm to (147.0, 120.5)
Routing:
- net GND: track 67.1 -> 59.2 mm
- net VCC: track 1160.0 -> 1155.1 mm
- net LED_AN: track 1568.5 -> 1564.0 mm
- net Net-(RGB2-Pad2): track 64.1 -> 67.7 mm
- net Net-(RGB4-Pad2): track 73.9 -> 76.7 mm
- net Net-(C8-Pad1): track 10.2 -> 12.7 mm
- net LED_CATH: track 1591.2 -> 1593.0 mm
- net Col8: track 255.9 -> 257.6 mm
- net Col2: track 113.1 -> 113.7 mm
- net Col5: track 113.7 -> 113.2 mm
