File: Kicad/DK60TP.kicad_pcb (KiCad board)
At the start: 2 copper layers, 285 x 113.5 mm, 336 parts, among them J1 USB_mini_micro_B, J2 RGB, J3 CAPS_LOCK, K0 K00, K10 K10, K100 K01, K110 K11, K120 K21, K130 K31, K140 K41, K141 K41, K142 K41, K20 K20, K200 K02, K21 K20, K210 K12, K220 K22, K230 K32, K240 K42, K241 K42, K30 K30, K300 K03, K31 K30, K310 K13, K320 K23, K330 K33, K340 LMB, K341 LMB, K40 K40, K400 K04, K41 K40, K410 K14, K420 K24, K430 K34, K440 MMB, K4C1 K4C, K500 K05, K510 K15, K520 K25, K530 K35, K540 K45, K600 K06, K610 K16, K620 K26, K630 K36, K640 K46, K641 K46, K642 K46, K643 K46, K700 K07, K710 K17, K720 K27, K730 K37, K740 K47, K800 K08, K810 K18, K820 K28, K830 K38, K840 RMB, K841 RMB, K900 K09, K910 K19, K920 K29, K930 K39, K940 K49, M1 MISC, M2 MISC, P1 MOUSE_BOARD, P2 MAIN_BOARD, P3 TRACKPOINT, SW1 RESET, U0 ATMEGA32U4-MU, U1 PAM2804, Y1 Crystal

Commit message: Updated wiring
Swap RGB and Row4 pins
Connections:
- U0 pad 26: Row4 -> RGB
- U0 pad 27: RGB -> Row4
Routing:
- net Row4: track 435.7 -> 449.9 mm
- net LED_AN: track 1564.0 -> 1554.5 mm
- net LED_CATH: track 1593.0 -> 1590.2 mm, vias 9 -> 10
- net Net-(DK14-Pad1): track 21.6 -> 24.4 mm
- net VCC: track 1155.1 -> 1152.7 mm
- net RGB: track 78.0 -> 76.2 mm
- net Net-(R2-Pad2): track 16.0 -> 17.1 mm
- net Col1: track 122.4 -> 123.5 mm
- net Col8: track 257.6 -> 256.9 mm, vias 8 -> 6
- net Col9: track 317.0 -> 316.5 mm, vias 6 -> 4

Commit message: Moved pin headers
Moved capslock pins, RGB extension plug and Mouse board plug
Parts:
- moved J2 48.7 mm to (201.2, 103.9), turned to 270 degrees
- moved J3 27.1 mm to (248.9, 121.1), turned to 180 degrees
- moved R6 11.1 mm to (235.2, 120.0), turned to 270 degrees
- moved DK74 3.23 mm to (223.7, 117.3)
- moved P1 1.00 mm to (211.0, 115.2)
Routing:
- net Net-(J3-Pad2): track 184.2 -> 220.6 mm
- net CAPS_LED: track 94.6 -> 111.2 mm
- net VCC: track 1152.7 -> 1168.6 mm, vias 21 -> 22
- net Col7: track 195.8 -> 184.6 mm, vias 4 -> 3
- net Net-(J3-Pad1): track 5.21 -> 13.8 mm
- net ColB: track 241.1 -> 245.7 mm
- net ColA: track 212.9 -> 208.3 mm
- net Row4: track 449.9 -> 446.0 mm
- net DOUT: track 134.9 -> 138.4 mm, vias 2 -> 1
- net LED_CATH: track 1590.2 -> 1587.4 mm
- net Col8: track 256.9 -> 255.2 mm, vias 6 -> 5
- net Net-(RGB4-Pad2): track 76.7 -> 75.1 mm
- net Net-(DK64-Pad1): track 42.7 -> 41.3 mm
- net D2: track 102.5 -> 103.4 mm
- net D5: track 103.6 -> 104.5 mm
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
Commit message: Removed some Vias
Parts:
- moved R6 1.20 mm to (236.4, 120.1), turned to 315 degrees
Routing:
- net LED_AN: track 1554.1 -> 1593.0 mm, vias 7 -> 5
- net LED_CATH: track 1587.4 -> 1596.3 mm, vias 10 -> 6
- net Net-(J3-Pad1): track 13.8 -> 12.2 mm
- net ColB: track 245.7 -> 246.4 mm
- net Net-(J3-Pad2): track 220.6 -> 221.3 mm

Commit message: Reduced VIAs quantity
Parts:
- moved J2 0.50 mm to (200.7, 103.9)
- moved J3 0.50 mm to (249.4, 121.1)
Routing:
- net Col4: track 226.4 -> 199.2 mm
- net Col3: track 240.7 -> 213.9 mm
- net LED_AN: track 1593.0 -> 1612.4 mm, vias 5 -> 2
- net Col7: track 184.6 -> 169.3 mm, vias 3 -> 2
- net Row3: track 341.4 -> 330.9 mm
- net LED_CATH: track 1596.3 -> 1588.0 mm, vias 6 -> 1
- net Net-(J3-Pad2): track 221.3 -> 215.2 mm
- net CAPS_LED: track 111.6 -> 109.5 mm
- net ColB: track 246.4 -> 244.4 mm
- net ColC: track 269.7 -> 271.0 mm
- net Net-(RGB0-Pad2): track 144.0 -> 142.9 mm
- net VCC: track 1168.6 -> 1167.9 mm
- net Row1: track 376.3 -> 376.8 mm

Commit message: Reduced useless VIAs quantity
Routing:
- net LED_AN: track 1612.4 -> 1616.7 mm, vias 2 -> 1

Commit message: Less than 100 VIAs!
Inverted col8 and col9 on Atmega to reduce the quantity of VIAs.
Parts:
- moved DK20 5.72 mm to (102.3, 46.7), turned to 225 degrees
- moved DK21 3.87 mm to (111.9, 62.0)
- moved DK22 2.77 mm to (116.4, 80.8)
- moved DK50 2.68 mm to (161.3, 44.4), turned to 225 degrees
- moved DK70 2.40 mm to (199.2, 43.1)
- moved DK6 2.15 mm to (180.3, 43.1)
Connections:
- U0 pad 39: Col8 -> Col9
- U0 pad 40: Col9 -> Col8
Routing:
- net Col9: track 316.5 -> 364.9 mm, vias 4 -> 2
- net Col8: track 255.2 -> 295.8 mm, vias 5 -> 3
- net LED_CATH: track 1588.0 -> 1580.0 mm
- net Row4: track 446.0 -> 438.1 mm
- net Col2: track 113.7 -> 107.3 mm, vias 4 -> 2
- net Net-(DK64-Pad1): track 41.3 -> 36.1 mm
- net Net-(DKD2-Pad1): track 31.8 -> 27.7 mm
- net Row0: track 399.2 -> 395.3 mm
- net VCC: track 1167.9 -> 1164.4 mm
- net LED_AN: track 1616.7 -> 1613.6 mm
- net Col5: track 113.2 -> 110.4 mm
- net Row2: track 354.1 -> 351.8 mm
- net Net-(DKD3-Pad1): track 26.6 -> 24.3 mm
- net Row3: track 330.9 -> 328.8 mm
- net Net-(KC0-Pad1): track 7.64 -> 5.82 mm
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
Commit message: Added 2 break holes and updated renders
* Added 2 break holes to increase solidity in case of the user wont
seperate the 2 parts
* Removed some 3D Shape to have a better render view
Parts:
- added M3: MISC, Footprint:BreakHoles_small, F.Cu at (156.4, 134.5)
- added M4: MISC, Footprint:BreakHoles_small, F.Cu at (251.3, 134.5)
- moved M1 0.06 mm to (63.8, 134.5)
Other:
- outline, holes or cut-outs redrawn

Commit message: Reduced VIAs
Parts:
- moved DK80 1.79 mm to (218.6, 42.8)
Routing:
- net Row4: track 438.1 -> 455.8 mm
- net LED_AN: track 1613.6 -> 1618.4 mm, vias 1 -> 0
- net D5: track 104.5 -> 108.1 mm
- net D2: track 103.4 -> 105.3 mm
- net ColD: track 291.5 -> 293.1 mm
- net ColB: track 244.4 -> 246.0 mm
- net ColA: track 207.8 -> 209.4 mm
- net RGB: track 76.2 -> 77.8 mm
- net ColC: track 271.2 -> 272.8 mm
- net VCC: track 1164.4 -> 1165.8 mm
- net Col8: track 295.8 -> 294.6 mm
- net Net-(DK80-Pad1): track 4.22 -> 4.95 mm
- net LED_CATH: track 1580.0 -> 1579.9 mm, vias 1 -> 0
